File: KICAD/KICAD.kicad_sch (KiCad schematic)
At the start: 522 parts, among them J11 Conn_01x04_Pin, J4 Conn_01x03_Pin, J5 Conn_01x03_Pin, U1 CD4066BE, U2 CD4066BE, U3 CD4066BE, U4 CD4066BE

Commit message: .
Parts:
- removed U1, U2, U3, U4: CD4066BE, Package_DIP:DIP-14_W7.62mm, symbol Analog_Switch:CD4066BE
- added C1000, C1001, C1002, C1003, C1004, C1005, C1006, C1007, C1008, C1009, C1010, C1011, C1012, C1013, C1014, C1015, C1016, C1017, C1018, C1019, C1020, C1021, C1022, C1023, C1024, C1025, C1026, C1027, C1028, C1029, C1030, C1031, C1032, C1033, C1034, C1035, C1036, C1037, C1038, C1039, C1040, C1041, C1042, C1043, C1044, C1045, C1046, C1047, C1048, C1049, C1050, C1051, C1052, C1053, C1054, C1055, C1056, C1057, C1058, C1059, C1060, C1061, C1062, C1063, C1064, C1065, C1066, C1067, C1068, C1069, C1070, C1071, C1072, C1073, C1074, C1075, C1076, C1077, C1078, C1079, C1080, C1081, C1082, C1083, C1084, C1085, C1086, C1087, C1088, C1089, C1090, C1091, C1092, C1093, C1094, C1095, C1096, C1097, C1098, C1099, C1100, C1101, C1102, C1103, C1104, C1105, C1106, C1107, C1108, C1109, C1110, C1111, C1112, C1113, C1114, C1115, C1116, C1117, C1118, C1119, C1120, C1121, C1122, C1123, C1124, C1125, C1126, C1127, C1128, C1129, C1130, C1131, C1132, C1133, C1134, C1135, C1136, C1137, C1138, C1139, C1140, C1141, C1142, C1143, C1144, C1145, C1146, C1147, C1148, C1149, C1150, C1151, C1152, C1153, C1154, C1155, C1156, C1157, C1158, C1159, C1160, C1161, C1162, C1163, C1164, C1165, C1166, C1167, C1168, C1169, C1170, C1171, C1172, C1173, C1174, C1175, C1176, C1177, C1178, C1179, C1180, C1181, C1182, C1183, C1184, C1185, C1186, C1187, C1188, C1189, C1190, C1191, C1192, C1193, C1194, C1195, C1196, C1197, C1198, C1199, C1200, C1201, C1202, C1203, C1204, C1205, C1206, C1207, C1208, C1209, C1210, C1211, C1212, C1213, C1214, C1215, C1216, C1217, C1218, C1219, C1220, C1221, C1222, C1223, C1224, C1225, C1226, C1227, C1228, C1229, C1230, C1231, C1232, C1233, C1234, C1235, C1236, C1237, C1238, C1239, C1240, C1241, C1242, C1243, C1244, C1245, C1246, C1247, C1248, C1249, C1250, C1251, C1252, C1253, C1254, C1255, C1256, C1257, C1258, C1259, C1260, C1261, C1262, C1263, C1264, C1265, C1266, C1267, C1268, C1269, C1270, C1271, C1272, C1273, C1274, C1275, C1276, C1277, C1278, C1279, C1280, C1281, C1282, C1283, C1284, C1285, C1286, C1287, C1288, C1289, C1290, C1291, C1292, C1293, C1294, C1295, C1296, C1297, C1298, C1299, C1300, C1301, C1302, C1303, C1304, C1305, C1306, C1307, C1308, C1309, C1310, C1311, C1312, C1313, C1314, C1315, C1316, C1317, C1318, C1319, C1320, C1321, C1322, C1323, C1324, C1325, C1326, C1327, C1328, C1329, C1330, C1331, C1332, C1333, C1334, C1335, C1336, C1337, C1338, C1339, C1340, C1341, C1342, C1343, C1344, C1345, C1346, C1347, C1348, C1349, C1350, C1351, C1352, C1353, C1354, C1355, C1356, C1357, C1358, C1359, C1360, C1361, C1362, C1363, C1364, C1365, C1366, C1367, C1368, C1369, C1370, C1371, C1372, C1373, C1374, C1375, C1376, C1377, C1378, C1379, C1380, C1381, C1382, C1383, C1384, C1385, C1386, C1387, C1388, C1389, C1390, C1391, C1392, C1393, C1394, C1395, C1396, C1397, C1398, C1399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: C_Small, symbol Device:C_Small
- added D1000, D1001, D1002, D1003, D1004, D1005, D1006, D1007, D1008, D1009, D1010, D1011, D1012, D1013, D1014, D1015, D1016, D1017, D1018, D1019, D1020, D1021, D1022, D1023, D1024, D1025, D1026, D1027, D1028, D1029, D1030, D1031, D1032, D1033, D1034, D1035, D1036, D1037, D1038, D1039, D1040, D1041, D1042, D1043, D1044, D1045, D1046, D1047, D1048, D1049, D1050, D1051, D1052, D1053, D1054, D1055, D1056, D1057, D1058, D1059, D1060, D1061, D1062, D1063, D1064, D1065, D1066, D1067, D1068, D1069, D1070, D1071, D1072, D1073, D1074, D1075, D1076, D1077, D1078, D1079, D1080, D1081, D1082, D1083, D1084, D1085, D1086, D1087, D1088, D1089, D1090, D1091, D1092, D1093, D1094, D1095, D1096, D1097, D1098, D1099, D1100, D1101, D1102, D1103, D1104, D1105, D1106, D1107, D1108, D1109, D1110, D1111, D1112, D1113, D1114, D1115, D1116, D1117, D1118, D1119, D1120, D1121, D1122, D1123, D1124, D1125, D1126, D1127, D1128, D1129, D1130, D1131, D1132, D1133, D1134, D1135, D1136, D1137, D1138, D1139, D1140, D1141, D1142, D1143, D1144, D1145, D1146, D1147, D1148, D1149, D1150, D1151, D1152, D1153, D1154, D1155, D1156, D1157, D1158, D1159, D1160, D1161, D1162, D1163, D1164, D1165, D1166, D1167, D1168, D1169, D1170, D1171, D1172, D1173, D1174, D1175, D1176, D1177, D1178, D1179, D1180, D1181, D1182, D1183, D1184, D1185, D1186, D1187, D1188, D1189, D1190, D1191, D1192, D1193, D1194, D1195, D1196, D1197, D1198, D1199, D1200, D1201, D1202, D1203, D1204, D1205, D1206, D1207, D1208, D1209, D1210, D1211, D1212, D1213, D1214, D1215, D1216, D1217, D1218, D1219, D1220, D1221, D1222, D1223, D1224, D1225, D1226, D1227, D1228, D1229, D1230, D1231, D1232, D1233, D1234, D1235, D1236, D1237, D1238, D1239, D1240, D1241, D1242, D1243, D1244, D1245, D1246, D1247, D1248, D1249, D1250, D1251, D1252, D1253, D1254, D1255, D1256, D1257, D1258, D1259, D1260, D1261, D1262, D1263, D1264, D1265, D1266, D1267, D1268, D1269, D1270, D1271, D1272, D1273, D1274, D1275, D1276, D1277, D1278, D1279, D1280, D1281, D1282, D1283, D1284, D1285, D1286, D1287, D1288, D1289, D1290, D1291, D1292, D1293, D1294, D1295, D1296, D1297, D1298, D1299, D1300, D1301, D1302, D1303, D1304, D1305, D1306, D1307, D1308, D1309, D1310, D1311, D1312, D1313, D1314, D1315, D1316, D1317, D1318, D1319, D1320, D1321, D1322, D1323, D1324, D1325, D1326, D1327, D1328, D1329, D1330, D1331, D1332, D1333, D1334, D1335, D1336, D1337, D1338, D1339, D1340, D1341, D1342, D1343, D1344, D1345, D1346, D1347, D1348, D1349, D1350, D1351, D1352, D1353, D1354, D1355, D1356, D1357, D1358, D1359, D1360, D1361, D1362, D1363, D1364, D1365, D1366, D1367, D1368, D1369, D1370, D1371, D1372, D1373, D1374, D1375, D1376, D1377, D1378, D1379, D1380, D1381, D1382, D1383, D1384, D1385, D1386, D1387, D1388, D1389, D1390, D1391, D1392, D1393, D1394, D1395, D1396, D1397, D1398, D1399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: WS2812B, LED_SMD:LED_WS2812B_PLCC4_5.0x5.0mm_P3.2mm, symbol LED:WS2812B
Connections:
- net GND: no longer C1.1, C10.1, C100.1, C101.1, C102.1, C103.1, C104.1, C105.1, C106.1, C107.1, C108.1, C109.1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
- net VCC_3: no longer C1.2, C10.2, C100.2, C101.2, C102.2, C103.2, C104.2, C105.2, C106.2, C107.2, C108.2, C109.2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
- net DOUT19: now reaches D209.4 (DIN)
- net DOUT19: now also D152.2 (DOUT)
- net at D184.2 (DOUT): no longer D185.4 (DIN)
- net DOUT2: now reaches D72.2 (DOUT)
- net DOUT2: now also D129.4 (DIN); no longer D73.4 (DIN)
- net DOUT18: now reaches D145.4 (DIN)
- net DOUT18: now also D88.2 (DOUT)
- net DIN3: now reaches D17.4 (DIN)
- net DOUT3: now reaches D193.4 (DIN)
- net DOUT3: now also D136.2 (DOUT)
- net DIN1: now reaches D1.4 (DIN)
- net DOUT10: now reaches D80.2 (DOUT)
- net DOUT10: now also D137.4 (DIN)
- net DOUT12: now reaches D208.2 (DOUT)
- net DOUT12: now also D265.4 (DIN)
- net DIN2: now reaches D9.4 (DIN)
- net DIN2: no longer D8.2 (DOUT)
- net DOUT11: now reaches D144.2 (DOUT)
- net DOUT11: now also D201.4 (DIN)
- net at D25.4 (DIN): no longer D24.2 (DOUT)
- net DOUT17: now reaches D81.4 (DIN)
- net DOUT17: now also D24.2 (DOUT)
- net at D169.4 (DIN): no longer D168.2 (DOUT)
- net at D217.4 (DIN): no longer D216.2 (DOUT)
- net at D89.4 (DIN): no longer D88.2 (DOUT)
- net DOUT1: now reaches D65.4 (DIN)
- net DOUT1: now also D8.2 (DOUT)
- net at D57.4 (DIN): no longer D56.2 (DOUT)
- net at D233.4 (DIN): no longer D232.2 (DOUT)
- net DOUT4: now reaches D200.2 (DOUT)
- net DOUT4: now also D257.4 (DIN); no longer D201.4 (DIN)
- net at D105.4 (DIN): no longer D104.2 (DOUT)
- net at D120.2 (DOUT): no longer D121.4 (DIN)
- net DOUT9: now reaches D16.2 (DOUT)
- net DOUT9: now also D73.4 (DIN)
- net at D40.2 (DOUT): no longer D41.4 (DIN)
- net at D153.4 (DIN): no longer D152.2 (DOUT)
- net at D248.2 (DOUT): no longer D249.4 (DIN)
- new net: C1126.2, D1126.1 (VDD)
- new net: D1126.2 (DOUT), D1127.4 (DIN)
- new net: C1190.1, D1126.3 (VSS)
- new net: D1125.2 (DOUT), D1126.4 (DIN)
- new net: C299.1, D236.3 (VSS)
- new net: C299.2, D300.1 (VDD)
- new net: C1178.1, D1114.3 (VSS)
- new net: C1178.2, D1178.1 (VDD)
- new net: C1132.1, D1068.3 (VSS)
- new net: C1132.2, D1132.1 (VDD)
- new net: C514.2, D515.1 (VDD)
- new net: C445.2, D446.1 (VDD)
- new net: D446.2 (DOUT), D447.4 (DIN)
- new net: C509.1, D446.3 (VSS)
- new net: D445.2 (DOUT), D446.4 (DIN)
- new net: C1221.2, D1221.1 (VDD)
- new net: D1221.2 (DOUT), D1222.4 (DIN)
- new net: C1285.1, D1221.3 (VSS)
- new net: D1220.2 (DOUT), D1221.4 (DIN)
- new net: C1053.2, D1053.1 (VDD)
- new net: C1133.1, D1069.3 (VSS)
- new net: C1133.2, D1133.1 (VDD)
- new net: C942.1, D879.3 (VSS)
- new net: C942.2, D943.1 (VDD)
- new net: C359.1, D296.3 (VSS)
- new net: C359.2, D360.1 (VDD)
- new net: C1406.1, D1342.3 (VSS)
- new net: C1406.2, D1406.1 (VDD)
- new net: C922.1, D859.3 (VSS)
- new net: C922.2, D923.1 (VDD)
- new net: C874.2, D875.1 (VDD)
- new net: D875.2 (DOUT), D876.4 (DIN)
- new net: C938.1, D875.3 (VSS)
- new net: D874.2 (DOUT), D875.4 (DIN)
- new net: C400.2, D401.1 (VDD)
- new net: D401.2 (DOUT), D402.4 (DIN)
- new net: C464.1, D401.3 (VSS)
- new net: C68.2, D69.1 (VDD)
- new net: C132.1, D69.3 (VSS)
- new net: C417.1, D354.3 (VSS)
- new net: C417.2, D418.1 (VDD)
- new net: C641.2, D642.1 (VDD)
- new net: D642.2 (DOUT), D643.4 (DIN)
- new net: C705.1, D642.3 (VSS)
- new net: D641.2 (DOUT), D642.4 (DIN)
- new net: C76.1, D13.3 (VSS)
- new net: C76.2, D77.1 (VDD)
- new net: C689.1, D626.3 (VSS)
- new net: C689.2, D690.1 (VDD)
- new net: C566.2, D567.1 (VDD)
- new net: D567.2 (DOUT), D568.4 (DIN)
- new net: C630.1, D567.3 (VSS)
- new net: D566.2 (DOUT), D567.4 (DIN)
- new net: C747.2, D748.1 (VDD)
- new net: D748.2 (DOUT), D749.4 (DIN)
- new net: C811.1, D748.3 (VSS)
- new net: D747.2 (DOUT), D748.4 (DIN)
- new net: C750.2, D751.1 (VDD)
- new net: D751.2 (DOUT), D752.4 (DIN)
- new net: C814.1, D751.3 (VSS)
- new net: D750.2 (DOUT), D751.4 (DIN)
- new net: C974.2, D975.1 (VDD)
- new net: D975.2 (DOUT), D976.4 (DIN)
- new net: D974.2 (DOUT), D975.4 (DIN)
- new net: C486.1, D423.3 (VSS)
- new net: C486.2, D487.1 (VDD)
- new net: C754.2, D755.1 (VDD)
- new net: D755.2 (DOUT), D756.4 (DIN)
- new net: C818.1, D755.3 (VSS)
- new net: D754.2 (DOUT), D755.4 (DIN)
- new net: C1430.1, D1366.3 (VSS)
- new net: C1430.2, D1430.1 (VDD)
- new net: C156.2, D157.1 (VDD)
- new net: C220.1, D157.3 (VSS)
- new net: C623.2, D624.1 (VDD)
- new net: C687.1, D624.3 (VSS)
- new net: D623.2 (DOUT), D624.4 (DIN)
- new net: C601.1, D538.3 (VSS)
- new net: C601.2, D602.1 (VDD)
- new net: C656.1, D593.3 (VSS)
- new net: C656.2, D657.1 (VDD)
- new net: C477.1, D414.3 (VSS)
- new net: C477.2, D478.1 (VDD)
- new net: C362.2, D363.1 (VDD)
- new net: D363.2 (DOUT), D364.4 (DIN)
- new net: C426.1, D363.3 (VSS)
- new net: D362.2 (DOUT), D363.4 (DIN)
- new net: C191.2, D192.1 (VDD)
- new net: C255.1, D192.3 (VSS)
- new net: C1427.1, D1363.3 (VSS)
- new net: C1427.2, D1427.1 (VDD)
- new net: C411.1, D348.3 (VSS)
- new net: C411.2, D412.1 (VDD)
- new net: C9.2, D10.1 (VDD)
- new net: C73.1, D10.3 (VSS)
- new net: C12.2, D13.1 (VDD)
- new net: C952.1, D889.3 (VSS)
- new net: C952.2, D953.1 (VDD)
- new net: C557.2, D558.1 (VDD)
- new net: D558.2 (DOUT), D559.4 (DIN)
- new net: C621.1, D558.3 (VSS)
- new net: D557.2 (DOUT), D558.4 (DIN)
- new net: C133.2, D134.1 (VDD)
- new net: C197.1, D134.3 (VSS)
- new net: C1082.2, D1082.1 (VDD)
- new net: C642.1, D579.3 (VSS)
- new net: C642.2, D643.1 (VDD)
- new net: C608.2, D609.1 (VDD)
- new net: D609.2 (DOUT), D610.4 (DIN)
- new net: C672.1, D609.3 (VSS)
- new net: C1513.1, D1449.3 (VSS)
- new net: C1513.2, D1513.1 (VDD)
- new net: C1120.2, D1120.1 (VDD)
- new net: C1184.1, D1120.3 (VSS)
- new net: D1119.2 (DOUT), D1120.4 (DIN)
- new net: C1360.1, D1296.3 (VSS)
- new net: C1360.2, D1360.1 (VDD)
- new net: C1352.1, D1288.3 (VSS)
- new net: C1352.2, D1352.1 (VDD)
- new net: C763.1, D700.3 (VSS)
- new net: C763.2, D764.1 (VDD)
- new net: C1514.2, D1514.1 (VDD)
- new net: D1514.2 (DOUT), D1515.4 (DIN)
- new net: D1513.2 (DOUT), D1514.4 (DIN)
- new net: C777.2, D778.1 (VDD)
- new net: D778.2 (DOUT), D779.4 (DIN)
- new net: C841.1, D778.3 (VSS)
- new net: D777.2 (DOUT), D778.4 (DIN)
- new net: C1414.2, D1414.1 (VDD)
- new net: D1414.2 (DOUT), D1415.4 (DIN)
- new net: C1478.1, D1414.3 (VSS)
- new net: D1413.2 (DOUT), D1414.4 (DIN)
- new net: C858.2, D859.1 (VDD)
- new net: D859.2 (DOUT), D860.4 (DIN)
- new net: D858.2 (DOUT), D859.4 (DIN)
- new net: C39.2, D40.1 (VDD)
- new net: C103.1, D40.3 (VSS)
- new net: C823.1, D760.3 (VSS)
- new net: C823.2, D824.1 (VDD)
- new net: C654.1, D591.3 (VSS)
- new net: C654.2, D655.1 (VDD)
- new net: C650.1, D587.3 (VSS)
- new net: C650.2, D651.1 (VDD)
- new net: C609.2, D610.1 (VDD)
- new net: D610.2 (DOUT), D611.4 (DIN)
- new net: C673.1, D610.3 (VSS)
- new net: C1183.1, D1119.3 (VSS)
- new net: C1183.2, D1183.1 (VDD)
- new net: C813.2, D814.1 (VDD)
- new net: D814.2 (DOUT), D815.4 (DIN)
- new net: C877.1, D814.3 (VSS)
- new net: D813.2 (DOUT), D814.4 (DIN)
- new net: C925.1, D862.3 (VSS)
- new net: C925.2, D926.1 (VDD)
- new net: C841.2, D842.1 (VDD)
- new net: D842.2 (DOUT), D843.4 (DIN)
- new net: C905.1, D842.3 (VSS)
- new net: D841.2 (DOUT), D842.4 (DIN)
- new net: C1364.2, D1364.1 (VDD)
- new net: D1364.2 (DOUT), D1365.4 (DIN)
- new net: C1428.1, D1364.3 (VSS)
- new net: D1363.2 (DOUT), D1364.4 (DIN)
- new net: C333.1, D270.3 (VSS)
- new net: C333.2, D334.1 (VDD)
- new net: C1433.2, D1433.1 (VDD)
- new net: D1433.2 (DOUT), D1434.4 (DIN)
- new net: C1497.1, D1433.3 (VSS)
- new net: C1207.1, D1143.3 (VSS)
- new net: C1207.2, D1207.1 (VDD)
- new net: C152.1, D89.3 (VSS)
- new net: C152.2, D153.1 (VDD)
- new net: C1050.2, D1050.1 (VDD)
- new net: C585.2, D586.1 (VDD)
- new net: D586.2 (DOUT), D587.4 (DIN)
- new net: C649.1, D586.3 (VSS)
- new net: D585.2 (DOUT), D586.4 (DIN)
- new net: C613.1, D550.3 (VSS)
- new net: C613.2, D614.1 (VDD)
- new net: C970.2, D971.1 (VDD)
- new net: D971.2 (DOUT), D972.4 (DIN)
- new net: D970.2 (DOUT), D971.4 (DIN)
- new net: C1378.2, D1378.1 (VDD)
- new net: D1378.2 (DOUT), D1379.4 (DIN)
- new net: C1442.1, D1378.3 (VSS)
- new net: D1377.2 (DOUT), D1378.4 (DIN)
- new net: C304.2, D305.1 (VDD)
- new net: D305.2 (DOUT), D306.4 (DIN)
- new net: C368.1, D305.3 (VSS)
- new net: C893.2, D894.1 (VDD)
- new net: D894.2 (DOUT), D895.4 (DIN)
- new net: C957.1, D894.3 (VSS)
- new net: D893.2 (DOUT), D894.4 (DIN)
- new net: C246.1, D183.3 (VSS)
- new net: C246.2, D247.1 (VDD)
- new net: C1209.2, D1209.1 (VDD)
- new net: D1209.2 (DOUT), D1210.4 (DIN)
- new net: C1273.1, D1209.3 (VSS)
- new net: C1342.2, D1342.1 (VDD)
- new net: D1342.2 (DOUT), D1343.4 (DIN)
- new net: D1341.2 (DOUT), D1342.4 (DIN)
- new net: C335.2, D336.1 (VDD)
- new net: C399.1, D336.3 (VSS)
- new net: D335.2 (DOUT), D336.4 (DIN)
- new net: C1099.2, D1099.1 (VDD)
- new net: D1099.2 (DOUT), D1100.4 (DIN)
- new net: C1163.1, D1099.3 (VSS)
- new net: D1098.2 (DOUT), D1099.4 (DIN)
- new net: C741.1, D678.3 (VSS)
- new net: C741.2, D742.1 (VDD)
- new net: C916.2, D917.1 (VDD)
- new net: D917.2 (DOUT), D918.4 (DIN)
- new net: C981.1, D917.3 (VSS)
- new net: D916.2 (DOUT), D917.4 (DIN)
- new net: C564.2, D565.1 (VDD)
- new net: D565.2 (DOUT), D566.4 (DIN)
- new net: C628.1, D565.3 (VSS)
- new net: D564.2 (DOUT), D565.4 (DIN)
- new net: C460.1, D397.3 (VSS)
- new net: C460.2, D461.1 (VDD)
- new net: C388.1, D325.3 (VSS)
- new net: C388.2, D389.1 (VDD)
- new net: C1163.2, D1163.1 (VDD)
- new net: C1487.2, D1487.1 (VDD)
- new net: D1487.2 (DOUT), D1488.4 (DIN)
- new net: D1486.2 (DOUT), D1487.4 (DIN)
- new net: C1061.2, D1061.1 (VDD)
- new net: C1259.2, D1259.1 (VDD)
- new net: D1259.2 (DOUT), D1260.4 (DIN)
- new net: C1323.1, D1259.3 (VSS)
- new net: D1258.2 (DOUT), D1259.4 (DIN)
- new net: C1233.2, D1233.1 (VDD)
- new net: D1233.2 (DOUT), D1234.4 (DIN)
- new net: C1297.1, D1233.3 (VSS)
- new net: C1182.2, D1182.1 (VDD)
- new net: D1182.2 (DOUT), D1183.4 (DIN)
- new net: C1246.1, D1182.3 (VSS)
- new net: D1181.2 (DOUT), D1182.4 (DIN)
- new net: C302.2, D303.1 (VDD)
- new net: D303.2 (DOUT), D304.4 (DIN)
- new net: C366.1, D303.3 (VSS)
- new net: D302.2 (DOUT), D303.4 (DIN)
- new net: C406.2, D407.1 (VDD)
- new net: D407.2 (DOUT), D408.4 (DIN)
- new net: C470.1, D407.3 (VSS)
- new net: D406.2 (DOUT), D407.4 (DIN)
- new net: C46.2, D47.1 (VDD)
- new net: C861.2, D862.1 (VDD)
- new net: D862.2 (DOUT), D863.4 (DIN)
- new net: D861.2 (DOUT), D862.4 (DIN)
- new net: C1164.1, D1100.3 (VSS)
- new net: C1164.2, D1164.1 (VDD)
- new net: C1466.1, D1402.3 (VSS)
- new net: C1466.2, D1466.1 (VDD)
- new net: C1455.2, D1455.1 (VDD)
- new net: D1455.2 (DOUT), D1456.4 (DIN)
- new net: C1519.1, D1455.3 (VSS)
- new net: D1454.2 (DOUT), D1455.4 (DIN)
- new net: C153.1, D90.3 (VSS)
- new net: C153.2, D154.1 (VDD)
- new net: C1004.1, D940.3 (VSS)
- new net: C1004.2, D1004.1 (VDD)
- new net: C487.2, D488.1 (VDD)
- new net: D487.2 (DOUT), D488.4 (DIN)
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Other:
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
Commit message: .
Parts:
- removed C10, C100, C1000, C1001, C1002, C1003, C1004, C1005, C1006, C1007, C1008, C1009, C101, C1010, C1011, C1012, C1013, C1014, C1015, C1016, C1017, C1018, C1019, C102, C1020, C1021, C1022, C1023, C1024, C1025, C1026, C1027, C1028, C1029, C103, C1030, C1031, C1032, C1033, C1034, C1035, C1036, C1037, C1038, C1039, C104, C1040, C1041, C1042, C1043, C1044, C1045, C1046, C1047, C1048, C1049, C105, C1050, C1051, C1052, C1053, C1054, C1055, C1056, C1057, C1058, C1059, C106, C1060, C1061, C1062, C1063, C1064, C1065, C1066, C1067, C1068, C1069, C107, C1070, C1071, C1072, C1073, C1074, C1075, C1076, C1077, C1078, C1079, C108, C1080, C1081, C1082, C1083, C1084, C1085, C1086, C1087, C1088, C1089, C109, C1090, C1091, C1092, C1093, C1094, C1095, C1096, C1097, C1098, C1099, C110, C1100, C1101, C1102, C1103, C1104, C1105, C1106, C1107, C1108, C1109, C111, C1110, C1111, C1112, C1113, C1114, C1115, C1116, C1117, C1118, C1119, C112, C1120, C1121, C1122, C1123, C1124, C1125, C1126, C1127, C1128, C1129, C113, C1130, C1131, C1132, C1133, C1134, C1135, C1136, C1137, C1138, C1139, C114, C1140, C1141, C1142, C1143, C1144, C1145, C1146, C1147, C1148, C1149, C115, C1150, C1151, C1152, C1153, C1154, C1155, C1156, C1157, C1158, C1159, C116, C1160, C1161, C1162, C1163, C1164, C1165, C1166, C1167, C1168, C1169, C117, C1170, C1171, C1172, C1173, C1174, C1175, C1176, C1177, C1178, C1179, C118, C1180, C1181, C1182, C1183, C1184, C1185, C1186, C1187, C1188, C1189, C119, C1190, C1191, C1192, C1193, C1194, C1195, C1196, C1197, C1198, C1199, C12, C120, C1200, C1201, C1202, C1203, C1204, C1205, C1206, C1207, C1208, C1209, C121, C1210, C1211, C1212, C1213, C1214, C1215, C1216, C1217, C1218, C1219, C122, C1220, C1221, C1222, C1223, C1224, C1225, C1226, C1227, C1228, C1229, C123, C1230, C1231, C1232, C1233, C1234, C1235, C1236, C1237, C1238, C1239, C124, C1240, C1241, C1242, C1243, C1244, C1245, C1246, C1247, C1248, C1249, C125, C1250, C1251, C1252, C1253, C1254, C1255, C1256, C1257, C1258, C1259, C126, C1260, C1261, C1262, C1263, C1264, C1265, C1266, C1267, C1268, C1269, C127, C1270, C1271, C1272, C1273, C1274, C1275, C1276, C1277, C1278, C1279, C128, C1280, C1281, C1282, C1283, C1284, C1285, C1286, C1287, C1288, C1289, C129, C1290, C1291, C1292, C1293, C1294, C1295, C1296, C1297, C1298, C1299, C13, C130, C1300, C1301, C1302, C1303, C1304, C1305, C1306, C1307, C1308, C1309, C131, C1310, C1311, C1312, C1313, C1314, C1315, C1316, C1317, C1318, C1319, C132, C1320, C1321, C1322, C1323, C1324, C1325, C1326, C1327, C1328, C1329, C133, C1330, C1331, C1332, C1333, C1334, C1335, C1336, C1337, C1338, C1339, C134, C1340, C1341, C1342, C1343, C1344, C1345, C1346, C1347, C1348, C1349, C135, C1350, C1351, C1352, C1353, C1354, C1355, C1356, C1357, C1358, C1359, C136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: C_Small, symbol Device:C_Small
- added C10, C12, C13, C15, C16, C18, C19, C21, C22, C3, C4, C6, C7, C9: 16PK4700MEFC12.5X25, Capacitor_THT:CP_Radial_D5.0mm_P2.50mm, symbol Device:C_Polarized
- added D1537, D1538, D1539, D1540, D1541, D1542, D1543, D1544, D1545, D1546, D1547, D1548, D1549, D1550, D1551, D1552, D1553, D1554, D1555, D1556, D1557, D1558, D1559, D1560, D1561, D1562, D1563, D1564, D1565, D1566, D1567, D1568, D1569, D1570, D1571, D1572, D1573, D1574, D1575, D1576, D1577, D1578, D1579, D1580, D1581, D1582, D1583, D1584, D1585, D1586, D1587, D1588, D1589, D1590, D1591, D1592, D1593, D1594, D1595, D1596, D1597, D1598, D1599, D1600, D1601, D1602, D1603, D1604, D1605, D1606, D1607, D1608, D1609, D1610, D1611, D1612, D1613, D1614, D1615, D1616, D1617, D1618, D1619, D1620, D1621, D1622, D1623, D1624, D1625, D1626, D1627, D1628, D1629, D1630, D1631, D1632, D1633, D1634, D1635, D1636, D1637, D1638, D1639, D1640, D1641, D1642, D1643, D1644, D1645, D1646, D1647, D1648, D1649, D1650, D1651, D1652, D1653, D1654, D1655, D1656, D1657, D1658, D1659, D1660, D1661, D1662, D1663, D1664, D1665, D1666, D1667, D1668, D1669, D1670, D1671, D1672, D1673, D1674, D1675, D1676, D1677, D1678, D1679, D1680, D1681, D1682, D1683, D1684, D1685, D1686, D1687, D1688, D1689, D1690, D1691, D1692, D1693, D1694, D1695, D1696, D1697, D1698, D1699, D1700, D1701, D1702, D1703, D1704, D1705, D1706, D1707, D1708, D1709, D1710, D1711, D1712, D1713, D1714, D1715, D1716, D1717, D1718, D1719, D1720, D1721, D1722, D1723, D1724, D1725, D1726, D1727, D1728, D1729, D1730, D1731, D1732, D1733, D1734, D1735, D1736, D1737, D1738, D1739, D1740, D1741, D1742, D1743, D1744, D1745, D1746, D1747, D1748, D1749, D1750, D1751, D1752, D1753, D1754, D1755, D1756, D1757, D1758, D1759, D1760, D1761, D1762, D1763, D1764, D1765, D1766, D1767, D1768, D1769, D1770, D1771, D1772, D1773, D1774, D1775, D1776, D1777, D1778, D1779, D1780, D1781, D1782, D1783, D1784, D1785, D1786, D1787, D1788, D1789, D1790, D1791, D1792, D1793, D1794, D1795, D1796, D1797, D1798, D1799, D1800, D1801, D1802, D1803, D1804, D1805, D1806, D1807, D1808, D1809, D1810, D1811, D1812, D1813, D1814, D1815, D1816, D1817, D1818, D1819, D1820, D1821, D1822, D1823, D1824, D1825, D1826, D1827, D1828, D1829, D1830, D1831, D1832, D1833, D1834, D1835, D1836, D1837, D1838, D1839, D1840, D1841, D1842, D1843, D1844, D1845, D1846, D1847, D1848, D1849, D1850, D1851, D1852, D1853, D1854, D1855, D1856, D1857, D1858, D1859, D1860, D1861, D1862, D1863, D1864, D1865, D1866, D1867, D1868, D1869, D1870, D1871, D1872, D1873, D1874, D1875, D1876, D1877, D1878, D1879, D1880, D1881, D1882, D1883, D1884, D1885, D1886, D1887, D1888, D1889, D1890, D1891, D1892, D1893, D1894, D1895, D1896, D1897, D1898, D1899, D1900, D1901, D1902, D1903, D1904, D1905, D1906, D1907, D1908, D1909, D1910, D1911, D1912, D1913, D1914, D1915, D1916, D1917, D1918, D1919, D1920, D1921, D1922, D1923, D1924, D1925, D1926, D1927, D1928, D1929, D1930, D1931, D1932, D1933, D1934, D1935, D1936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: WS2812B, LED_SMD:LED_WS2812B_PLCC4_5.0x5.0mm_P3.2mm, symbol LED:WS2812B
- added U1: STM32G070RBTx, Package_QFP:LQFP-64_10x10mm_P0.5mm, symbol MCU_ST_STM32G0:STM32G070RBTx
- added U2: AMS1117-3.3, Package_TO_SOT_SMD:SOT-223-3_TabPin2, symbol Regulator_Linear:AMS1117-3.3
- C1: footprint (none) -> Capacitor_SMD:C_0603_1608Metric
- C11, C14, C17, C2, C20, C5, C8: value C_Small -> T520Y337M006ATE040; footprint (none) -> Capacitor_SMD:CP_Elec_10x10
- C23, C24, C25, C26: value C_Small -> 0.1
- C27: value C_Small -> 2.2
Connections:
- net DOUT16 is gone; now on an unnamed net: D464.2 (DOUT)
- net DOUT24 is gone; now on an unnamed net: D472.2 (DOUT)
- net DOUT8 is gone; now on an unnamed net: D456.2 (DOUT)
- net GND: now also C1.1, C11.2, C14.2, C17.2, C2.2, C20.2, C23.2, C24.2, C25.2, C26.2, C27.2, C5.2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
- net VCC_3: now also C1.2, C11.1, C14.1, C17.1, C2.1, C20.1, C23.1, C24.1, C25.1, C26.1, C27.1, C5.1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
- net at D1127.4 (DIN): now also D1128.2 (DOUT); no longer D1126.2 (DOUT)
- net at D1125.2 (DOUT): now also D1124.4 (DIN); no longer D1126.4 (DIN)
- net at D1222.4 (DIN): now also D1223.2 (DOUT); no longer D1221.2 (DOUT)
- net at D1220.2 (DOUT): now also D1219.4 (DIN); no longer D1221.4 (DIN)
- net at D876.4 (DIN): now also D877.2 (DOUT); no longer D875.2 (DOUT)
- net at D875.4 (DIN): now also D876.2 (DOUT); no longer D874.2 (DOUT)
- net at D70.4 (DIN): now also D71.2 (DOUT); no longer D69.2 (DOUT)
- net at D68.2 (DOUT): now also D67.4 (DIN); no longer D69.4 (DIN)
- net at D748.2 (DOUT): now also D747.4 (DIN); no longer D749.4 (DIN)
- net at D748.4 (DIN): now also D749.2 (DOUT); no longer D747.2 (DOUT)
- net at D751.2 (DOUT): now also D750.4 (DIN); no longer D752.4 (DIN)
- net at D750.2 (DOUT): now also D749.4 (DIN); no longer D751.4 (DIN)
- net at D976.4 (DIN): now also D912.2 (DOUT); no longer D975.2 (DOUT)
- net at D975.4 (DIN): now also D976.2 (DOUT); no longer D974.2 (DOUT)
- net at D755.2 (DOUT): now also D754.4 (DIN); no longer D756.4 (DIN)
- net at D754.2 (DOUT): now also D753.4 (DIN); no longer D755.4 (DIN)
- net at D624.2 (DOUT): now also D623.4 (DIN)
- net at D624.4 (DIN): now also D560.2 (DOUT); no longer D623.2 (DOUT)
- net at D364.4 (DIN): now also D365.2 (DOUT); no longer D363.2 (DOUT)
- net at D362.2 (DOUT): now also D361.4 (DIN); no longer D363.4 (DIN)
- net at D192.1 (VDD): now also D256.1 (VDD)
- net at D192.2 (DOUT): now also D256.4 (DIN)
- net at D609.2 (DOUT): now also D673.4 (DIN); no longer D610.4 (DIN)
- net at D609.4 (DIN): now also D610.2 (DOUT)
- net at D1120.2 (DOUT): now also D1119.4 (DIN)
- net at D1119.2 (DOUT): now also D1118.4 (DIN); no longer D1120.4 (DIN)
- net at D1515.4 (DIN): now also D1516.2 (DOUT); no longer D1514.2 (DOUT)
- net at D1514.4 (DIN): now also D1515.2 (DOUT); no longer D1513.2 (DOUT)
- net at D860.4 (DIN): now also D861.2 (DOUT); no longer D859.2 (DOUT)
- net at D859.4 (DIN): now also D860.2 (DOUT); no longer D858.2 (DOUT)
- net at D40.2 (DOUT): now also D104.4 (DIN)
- net at D611.4 (DIN): now also D612.2 (DOUT); no longer D610.2 (DOUT)
- net at D842.2 (DOUT): now also D841.4 (DIN); no longer D843.4 (DIN)
- net at D841.2 (DOUT): now also D905.4 (DIN); no longer D842.4 (DIN)
- net at D1365.4 (DIN): now also D1366.2 (DOUT); no longer D1364.2 (DOUT)
- net at D1363.2 (DOUT): now also D1362.4 (DIN); no longer D1364.4 (DIN)
- net at D1433.4 (DIN): now also D1369.2 (DOUT)
- net at D587.4 (DIN): now also D588.2 (DOUT); no longer D586.2 (DOUT)
- net at D586.4 (DIN): now also D587.2 (DOUT); no longer D585.2 (DOUT)
- net at D971.2 (DOUT): now also D970.4 (DIN); no longer D972.4 (DIN)
- net at D971.4 (DIN): now also D972.2 (DOUT); no longer D970.2 (DOUT)
- net at D1379.4 (DIN): now also D1380.2 (DOUT); no longer D1378.2 (DOUT)
- net at D1378.4 (DIN): now also D1379.2 (DOUT); no longer D1377.2 (DOUT)
- net at D305.4 (DIN): now also D241.2 (DOUT)
- net at D895.4 (DIN): now also D896.2 (DOUT); no longer D894.2 (DOUT)
- net at D893.2 (DOUT): now also D892.4 (DIN); no longer D894.4 (DIN)
- net at D1209.4 (DIN): now also D1145.2 (DOUT)
- net at D335.2 (DOUT): now also D334.4 (DIN); no longer D336.4 (DIN)
- net at D1099.2 (DOUT): now also D1098.4 (DIN); no longer D1100.4 (DIN)
- net at D1098.2 (DOUT): now also D1097.4 (DIN); no longer D1099.4 (DIN)
- net at D1488.4 (DIN): now also D1424.2 (DOUT); no longer D1487.2 (DOUT)
- net at D1486.2 (DOUT): now also D1485.4 (DIN); no longer D1487.4 (DIN)
- net at D1259.2 (DOUT): now also D1258.4 (DIN); no longer D1260.4 (DIN)
- net at D1259.4 (DIN): now also D1260.2 (DOUT); no longer D1258.2 (DOUT)
- net at D1233.2 (DOUT): now also D1297.4 (DIN); no longer D1234.4 (DIN)
- net at D1233.4 (DIN): now also D1234.2 (DOUT)
- net at D862.2 (DOUT): now also D861.4 (DIN); no longer D863.4 (DIN)
- net at D862.4 (DIN): now also D863.2 (DOUT); no longer D861.2 (DOUT)
- net at D1402.3 (VSS): now also D1401.3 (VSS), D1403.3 (VSS), D1404.3 (VSS), D1405.3 (VSS), D1406.3 (VSS), D1407.3 (VSS), D1408.3 (VSS), D1465.3 (VSS), D1466.3 (VSS), D1467.3 (VSS), D1468.3 (VSS), D1469.3 (VSS)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
- net at D488.2 (DOUT): now also D487.4 (DIN)
- net at D488.4 (DIN): now also D424.2 (DOUT); no longer D487.2 (DOUT)
- net at D409.4 (DIN): now also D345.2 (DOUT)
- net at D505.2 (DOUT): no longer D506.4 (DIN)
- net at D505.4 (DIN): now also D506.2 (DOUT)
- net at D234.4 (DIN): now also D235.2 (DOUT); no longer D233.2 (DOUT)
- removed net DOUT1: D65.4 (DIN), D8.2 (DOUT)
- removed net DOUT10: D137.4 (DIN), D80.2 (DOUT)
- removed net DOUT11: D144.2 (DOUT), D201.4 (DIN)
- removed net DOUT12: D208.2 (DOUT), D265.4 (DIN)
- removed net DOUT14: D336.2 (DOUT), D393.4 (DIN)
- removed net DOUT17: D24.2 (DOUT), D81.4 (DIN)
- removed net DOUT18: D145.4 (DIN), D88.2 (DOUT)
- removed net DOUT2: D129.4 (DIN), D72.2 (DOUT)
- removed net DOUT20: D216.2 (DOUT), D273.4 (DIN)
- removed net DOUT21: D280.2 (DOUT), D337.4 (DIN)
- removed net DOUT23: D408.2 (DOUT), D465.4 (DIN)
- removed net DOUT3: D136.2 (DOUT), D193.4 (DIN)
- removed net DOUT6: D328.2 (DOUT), D385.4 (DIN)
- removed net DOUT9: D16.2 (DOUT), D73.4 (DIN)
- new net: D1897.2 (DOUT), D1961.4 (DIN)
- new net: D1897.4 (DIN), D1898.2 (DOUT)
- new net: D1550.2 (DOUT), D1551.4 (DIN)
- new net: D1549.2 (DOUT), D1550.4 (DIN)
- new net: D1772.4 (DIN), D1773.2 (DOUT)
- new net: D1773.4 (DIN), D1774.2 (DOUT)
- new net: D3360.2 (DOUT), D3424.4 (DIN)
- new net: D3359.2 (DOUT), D3360.4 (DIN)
- new net: D2919.4 (DIN), D2920.2 (DOUT)
- new net: D2856.2 (DOUT), D2920.4 (DIN)
- new net: D2300.4 (DIN), D2301.2 (DOUT)
- new net: D2301.4 (DIN), D2302.2 (DOUT)
- new net: D2328.2 (DOUT), D2392.4 (DIN)
- new net: D2327.2 (DOUT), D2328.4 (DIN)
- new net: D1713.2 (DOUT), D1714.4 (DIN)
- new net: D1649.2 (DOUT), D1713.4 (DIN)
- new net: D2270.4 (DIN), D2271.2 (DOUT)
- new net: D2271.4 (DIN), D2272.2 (DOUT)
- new net: D2153.2 (DOUT), D2217.4 (DIN)
- new net: D2153.4 (DIN), D2154.2 (DOUT)
- new net: D3158.4 (DIN), D3159.2 (DOUT)
- new net: D3159.4 (DIN), D3160.2 (DOUT)
- new net: D2777.2 (DOUT), D2841.4 (DIN)
- new net: D2777.4 (DIN), D2778.2 (DOUT)
- new net: D1739.4 (DIN), D1740.2 (DOUT)
- new net: D1740.4 (DIN), D1741.2 (DOUT)
- new net: D1714.2 (DOUT), D1715.4 (DIN)
- new net: D3581.4 (DIN), D3582.2 (DOUT)
- new net: D3582.4 (DIN), D3583.2 (DOUT)
- new net: D3273.4 (DIN), D3274.2 (DOUT)
- new net: D3274.4 (DIN), D3275.2 (DOUT)
- new net: D2180.2 (DOUT), D2181.4 (DIN)
- new net: D2179.2 (DOUT), D2180.4 (DIN)
- new net: D3134.2 (DOUT), D3135.4 (DIN)
- new net: D3066.3 (VSS), D3067.3 (VSS), D3068.3 (VSS), D3069.3 (VSS), D3070.3 (VSS), D3071.3 (VSS), D3072.3 (VSS), D3130.3 (VSS), D3131.3 (VSS), D3132.3 (VSS), D3133.3 (VSS), D3134.3 (VSS)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
- new net: D3133.2 (DOUT), D3134.4 (DIN)
- new net: D1711.2 (DOUT), D1712.4 (DIN)
- new net: D1710.2 (DOUT), D1711.4 (DIN)
- new net: D1675.2 (DOUT), D1676.4 (DIN)
- new net: D1674.2 (DOUT), D1675.4 (DIN)
- new net: D3444.4 (DIN), D3445.2 (DOUT)
- new net: D3445.4 (DIN), D3446.2 (DOUT)
- new net: D2847.2 (DOUT), D2848.4 (DIN)
- new net: D2846.2 (DOUT), D2847.4 (DIN)
- new net: D2447.2 (DOUT), D2448.4 (DIN)
- new net: D2446.2 (DOUT), D2447.4 (DIN)
- new net: D3060.4 (DIN), D3061.2 (DOUT)
- new net: D3061.4 (DIN), D3062.2 (DOUT)
- new net: D1725.2 (DOUT), D1726.4 (DIN)
- new net: D1724.2 (DOUT), D1725.4 (DIN)
- new net: D1816.2 (DOUT), D1880.4 (DIN)
- new net: D1815.2 (DOUT), D1816.4 (DIN)
- new net: D1863.4 (DIN), D1864.2 (DOUT)
- new net: D1800.2 (DOUT), D1864.4 (DIN)
- new net: D3313.4 (DIN), D3314.2 (DOUT)
- new net: D3314.4 (DIN), D3315.2 (DOUT)
- new net: D1873.4 (DIN), D1874.2 (DOUT)
- new net: D1874.4 (DIN), D1875.2 (DOUT)
- new net: D3332.2 (DOUT), D3333.4 (DIN)
- new net: D3331.2 (DOUT), D3332.4 (DIN)
- new net: D2076.2 (DOUT), D2077.4 (DIN)
- new net: D2075.2 (DOUT), D2076.4 (DIN)
- new net: D2022.4 (DIN), D2023.2 (DOUT)
- new net: D2023.4 (DIN), D2024.2 (DOUT)
- new net: D1820.2 (DOUT), D1821.4 (DIN)
- new net: D1819.2 (DOUT), D1820.4 (DIN)
- new net: D2204.2 (DOUT), D2205.4 (DIN)
- new net: D2203.2 (DOUT), D2204.4 (DIN)
- new net: D2754.4 (DIN), D2755.2 (DOUT)
- new net: D2755.4 (DIN), D2756.2 (DOUT)
- new net: D1814.2 (DOUT), D1815.4 (DIN)
- new net: D3340.2 (DOUT), D3341.4 (DIN)
- new net: D3339.2 (DOUT), D3340.4 (DIN)
- new net: D2679.4 (DIN), D2680.2 (DOUT)
- new net: D2616.2 (DOUT), D2680.4 (DIN)
- new net: D2593.2 (DOUT), D2594.4 (DIN)
- new net: D1862.4 (DIN), D1863.2 (DOUT)
- new net: D3557.4 (DIN), D3558.2 (DOUT)
- new net: D3558.4 (DIN), D3559.2 (DOUT)
- new net: D2694.2 (DOUT), D2695.4 (DIN)
- new net: D2693.2 (DOUT), D2694.4 (DIN)
- new net: D2691.2 (DOUT), D2692.4 (DIN)
- new net: D2690.2 (DOUT), D2691.4 (DIN)
- new net: D2064.2 (DOUT), D2128.4 (DIN)
- new net: D2063.2 (DOUT), D2064.4 (DIN)
- new net: D1953.2 (DOUT), D1954.4 (DIN)
- new net: D1889.2 (DOUT), D1953.4 (DIN)
- new net: D1952.2 (DOUT), D2016.4 (DIN)
- new net: D1951.2 (DOUT), D1952.4 (DIN)
- new net: D2414.4 (DIN), D2415.2 (DOUT)
- new net: D2415.4 (DIN), D2416.2 (DOUT)
- new net: D1889.4 (DIN), D1890.2 (DOUT)
- new net: D2206.2 (DOUT), D2207.4 (DIN)
- new net: D2205.2 (DOUT), D2206.4 (DIN)
- new net: D1673.2 (DOUT), D1674.4 (DIN)
- new net: D1609.2 (DOUT), D1673.4 (DIN)
- new net: D2549.4 (DIN), D2550.2 (DOUT)
- new net: D2550.4 (DIN), D2551.2 (DOUT)
- new net: D3271.4 (DIN), D3272.2 (DOUT)
- new net: D3208.2 (DOUT), D3272.4 (DIN)
- new net: D3441.2 (DOUT), D3505.4 (DIN)
- new net: D3441.4 (DIN), D3442.2 (DOUT)
- new net: D1957.2 (DOUT), D1958.4 (DIN)
- new net: D1956.2 (DOUT), D1957.4 (DIN)
- new net: D1630.4 (DIN), D1631.2 (DOUT)
- new net: D1631.4 (DIN), D1632.2 (DOUT)
- new net: D2228.2 (DOUT), D2229.4 (DIN)
- new net: D2227.2 (DOUT), D2228.4 (DIN)
- new net: D2407.4 (DIN), D2408.2 (DOUT)
- new net: D2344.2 (DOUT), D2408.4 (DIN)
- new net: D2397.4 (DIN), D2398.2 (DOUT)
- new net: D2398.4 (DIN), D2399.2 (DOUT)
- new net: D1598.2 (DOUT), D1599.4 (DIN)
- new net: D1597.2 (DOUT), D1598.4 (DIN)
- new net: D1596.2 (DOUT), D1597.4 (DIN)
- new net: D1919.4 (DIN), D1920.2 (DOUT)
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Other:
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
Commit message: .
Parts:
- removed C17, C20: T520Y337M006ATE040, Capacitor_SMD:CP_Elec_10x10, symbol Device:C_Small
- removed C18, C19, C21, C22: 16PK4700MEFC12.5X25, Capacitor_THT:CP_Radial_D5.0mm_P2.50mm, symbol Device:C_Polarized
- removed C23, C24, C25, C26: 0.1, symbol Device:C_Small
- removed C27: 2.2, symbol Device:C_Small
- removed D1009, D1010, D1011, D1012, D1013, D1014, D1015, D1016, D1017, D1018, D1019, D1020, D1021, D1022, D1023, D1024, D1073, D1074, D1075, D1076, D1077, D1078, D1079, D1080, D1081, D1082, D1083, D1084, D1085, D1086, D1087, D1088, D113, D1137, D1138, D1139, D114, D1140, D1141, D1142, D1143, D1144, D1145, D1146, D1147, D1148, D1149, D115, D1150, D1151, D1152, D116, D117, D118, D119, D120, D1201, D1202, D1203, D1204, D1205, D1206, D1207, D1208, D1209, D121, D1210, D1211, D1212, D1213, D1214, D1215, D1216, D122, D123, D124, D125, D126, D1265, D1266, D1267, D1268, D1269, D127, D1270, D1271, D1272, D1273, D1274, D1275, D1276, D1277, D1278, D1279, D128, D1280, D1329, D1330, D1331, D1332, D1333, D1334, D1335, D1336, D1337, D1338, D1339, D1340, D1341, D1342, D1343, D1344, D1393, D1394, D1395, D1396, D1397, D1398, D1399, D1400, D1401, D1402, D1403, D1404, D1405, D1406, D1407, D1408, D1457, D1458, D1459, D1460, D1461, D1462, D1463, D1464, D1465, D1466, D1467, D1468, D1469, D1470, D1471, D1472, D1521, D1522, D1523, D1524, D1525, D1526, D1527, D1528, D1529, D1530, D1531, D1532, D1533, D1534, D1535, D1536, D1585, D1586, D1587, D1588, D1589, D1590, D1591, D1592, D1593, D1594, D1595, D1596, D1597, D1598, D1599, D1600, D1649, D1650, D1651, D1652, D1653, D1654, D1655, D1656, D1657, D1658, D1659, D1660, D1661, D1662, D1663, D1664, D1713, D1714, D1715, D1716, D1717, D1718, D1719, D1720, D1721, D1722, D1723, D1724, D1725, D1726, D1727, D1728, D177, D1777, D1778, D1779, D178, D1780, D1781, D1782, D1783, D1784, D1785, D1786, D1787, D1788, D1789, D179, D1790, D1791, D1792, D180, D181, D182, D183, D184, D1841, D1842, D1843, D1844, D1845, D1846, D1847, D1848, D1849, D185, D1850, D1851, D1852, D1853, D1854, D1855, D1856, D186, D187, D188, D189, D190, D1905, D1906, D1907, D1908, D1909, D191, D1910, D1911, D1912, D1913, D1914, D1915, D1916, D1917, D1918, D1919, D192, D1920, D1969, D1970, D1971, D1972, D1973, D1974, D1975, D1976, D1977, D1978, D1979, D1980, D1981, D1982, D1983, D1984, D2033, D2034, D2035, D2036, D2037, D2038, D2039, D2040, D2041, D2042, D2043, D2044, D2045, D2046, D2047, D2048, D2097, D2098, D2099, D2100, D2101, D2102, D2103, D2104, D2105, D2106, D2107, D2108, D2109, D2110, D2111, D2112, D2161, D2162, D2163, D2164, D2165, D2166, D2167, D2168, D2169, D2170, D2171, D2172, D2173, D2174, D2175, D2176, D2225, D2226, D2227, D2228, D2229, D2230, D2231, D2232, D2233, D2234, D2235, D2236, D2237, D2238, D2239, D2240, D2289, D2290, D2291, D2292, D2293, D2294, D2295, D2296, D2297, D2298, D2299, D2300, D2301, D2302, D2303, D2304, D2353, D2354, D2355, D2356, D2357, D2358, D2359, D2360, D2361, D2362, D2363, D2364, D2365, D2366, D2367, D2368, D241, D2417, D2418, D2419, D242, D2420, D2421, D2422, D2423, D2424, D2425, D2426, D2427, D2428, D2429, D243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: WS2812B, LED_SMD:LED_WS2812B_PLCC4_5.0x5.0mm_P3.2mm, symbol LED:WS2812B
- removed J11: Conn_01x04_Pin, Connector_PinHeader_2.54mm:PinHeader_1x04_P2.54mm_Horizontal, symbol Connector:Conn_01x04_Pin
- removed J4, J5: Conn_01x03_Pin, Connector_PinHeader_2.54mm:PinHeader_1x03_P2.54mm_Vertical, symbol Connector:Conn_01x03_Pin
- removed U1: STM32G070RBTx, Package_QFP:LQFP-64_10x10mm_P0.5mm, symbol MCU_ST_STM32G0:STM32G070RBTx
- removed U2: AMS1117-3.3, Package_TO_SOT_SMD:SOT-223-3_TabPin2, symbol Regulator_Linear:AMS1117-3.3
- added J3: Conn_02x20_Odd_Even, Connector_IDC:IDC-Header_2x20_P2.54mm_Vertical_SMD, symbol Connector_Generic:Conn_02x20_Odd_Even
- added J4: Conn_01x02_Pin, Connector_JST:JST_EH_B2B-EH-A_1x02_P2.50mm_Vertical, symbol Connector:Conn_01x02_Pin
- added J5: PJ-102A, digikey-footprints:Barrel_Jack_5.5mmODx2.1mmID_PJ-102A, symbol dk_Barrel-Power-Connectors:PJ-102A
- added R31: 10k, Resistor_SMD:R_0402_1005Metric, symbol Device:R
Connections:
- net GND: now also J3.37 (Pin_37), J3.38 (Pin_38), J3.39 (Pin_39), J3.40 (Pin_40), J5.2, J5.3
- net VCC_3: now also J5.1
- net BURST_F5: now reaches D2593.4 (DIN)
- net BURST_F5: now also J3.35 (Pin_35)
- net BURST_F6: now reaches D2601.4 (DIN)
- net BURST_F6: now also J3.36 (Pin_36)
- net BURST_E3: now reaches D2065.4 (DIN)
- net BURST_E3: now also J3.27 (Pin_27)
- net BURST_D1: now reaches D1537.4 (DIN)
- net BURST_D1: now also J3.19 (Pin_19)
- net BURST_A1: now reaches D1.4 (DIN)
- net BURST_A1: now also J3.1 (Pin_1)
- net BURST_C5: now reaches D1057.4 (DIN)
- net BURST_C5: now also J3.17 (Pin_17)
- net BURST_A6: now reaches D41.4 (DIN)
- net BURST_A6: now also J3.6 (Pin_6)
- net BURST_A3: now reaches D17.4 (DIN)
- net BURST_A3: now also J3.3 (Pin_3)
- net BURST_B1: now reaches D513.4 (DIN)
- net BURST_B1: now also J3.7 (Pin_7)
- net BURST_B3: now reaches D529.4 (DIN)
- net BURST_B3: now also J3.9 (Pin_9)
- net BURST_A5: now reaches D33.4 (DIN)
- net BURST_A5: now also J3.5 (Pin_5)
- net BURST_B4: now reaches D537.4 (DIN)
- net BURST_B4: now also J3.10 (Pin_10)
- net BURST_F2: now reaches D2569.4 (DIN)
- net BURST_F2: now also J3.32 (Pin_32)
- net BURST_F4: now reaches D2585.4 (DIN)
- net BURST_F4: now also J3.34 (Pin_34)
- net BURST_C2: now reaches D1033.4 (DIN)
- net BURST_C2: now also J3.14 (Pin_14)
- net BURST_E5: now reaches D2081.4 (DIN)
- net BURST_E5: now also J3.29 (Pin_29)
- net BURST_F3: now reaches D2577.4 (DIN)
- net BURST_F3: now also J3.33 (Pin_33)
- net BURST_C3: now reaches D1041.4 (DIN)
- net BURST_C3: now also J3.15 (Pin_15)
- net BURST_E4: now reaches D2073.4 (DIN)
- net BURST_E4: now also J3.28 (Pin_28)
- net BURST_B6: now reaches D553.4 (DIN)
- net BURST_B6: now also J3.12 (Pin_12)
- net BURST_C4: now reaches D1049.4 (DIN)
- net BURST_C4: now also J3.16 (Pin_16)
- net BURST_D6: now reaches D1577.4 (DIN)
- net BURST_D6: now also J3.24 (Pin_24)
- net BURST_B5: now reaches D545.4 (DIN)
- net BURST_B5: now also J3.11 (Pin_11)
- net BURST_C6: now reaches D1065.4 (DIN)
- net BURST_C6: now also J3.18 (Pin_18)
- net BURST_C1: now reaches D1025.4 (DIN)
- net BURST_C1: now also J3.13 (Pin_13)
- net BURST_D5: now reaches D1569.4 (DIN)
- net BURST_D5: now also J3.23 (Pin_23)
- net BURST_D4: now reaches D1561.4 (DIN)
- net BURST_D4: now also J3.22 (Pin_22)
- net BURST_A2: now reaches D9.4 (DIN)
- net BURST_A2: now also J3.2 (Pin_2)
- net BURST_D3: now reaches D1553.4 (DIN)
- net BURST_D3: now also J3.21 (Pin_21)
- net BURST_E2: now reaches D2057.4 (DIN)
- net BURST_E2: now also J3.26 (Pin_26)
- net BURST_F1: now reaches D2561.4 (DIN)
- net BURST_F1: now also J3.31 (Pin_31)
- net BURST_B2: now reaches D521.4 (DIN)
- net BURST_B2: now also J3.8 (Pin_8)
- net BURST_E6: now reaches D2089.4 (DIN)
- net BURST_E6: now also J3.30 (Pin_30)
- net BURST_E1: now reaches D2049.4 (DIN)
- net BURST_E1: now also J3.25 (Pin_25)
- net BURST_A4: now reaches D25.4 (DIN)
- net BURST_A4: now also J3.4 (Pin_4)
- net BURST_D2: now reaches D1545.4 (DIN)
- net BURST_D2: now also J3.20 (Pin_20)
- new net: J4.2 (Pin_2), R31.2
- new net STM_SIGNAL: J4.1 (Pin_1)
- new net VCC_3.3V: R31.1
- no-connect marks 56 -> 36
Other:
- moved on the sheet: C10, C11, C12, C13, C14, C15, C16, C2, C3, C4, C4210, C4211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
