File: stm/ws2812b_module/kicad/kicad.kicad_pcb (KiCad board)
At the start: 2 copper layers, 85 parts, among them J12 USB_ASP, J4 Conn_02x25_Odd_Even, J5 Conn_02x25_Odd_Even, J6 Conn_02x25_Odd_Even, J7 Conn_02x25_Odd_Even, Q1 T2N7002AK, Q2 T2N7002AK, Q3 T2N7002AK, Q4 T2N7002AK, SW1 SW_Push, SW2 SW_Push, SW3 SW_Push, U1 FXMA108, U10 FXMA108, U11 FXMA108, U12 AMS1117-3.3, U13 FXMA108, U14 74CBT16210CDGG, U16 74CBT16210CDGG, U17 74CBT16210CDGG, U2 FXMA108, U3 FXMA108, U4 FXMA108, U5 FXMA108, U6 STM32H563VGTx, U7 ATmega328-A, U8 FXMA108, U9 FXMA108, Y1 26MHz, Y2 Crystal

Commit message: .
Parts:
- removed J6, J7: Conn_02x25_Odd_Even, Connector_IDC:IDC-Header_2x25_P2.54mm_Vertical_SMD
- removed U2, U3, U4: FXMA108, Package_DFN_QFN:WQFN-20-1EP_2.5x4.5mm_P0.5mm_EP1x2.9mm
- added J1: Conn_01x03_Pin, Connector_JST:JST_EH_B3B-EH-A_1x03_P2.50mm_Vertical, F.Cu at (-135.6, 43.3)
- added J10: Conn_02x25_Odd_Even, Connector_IDC:IDC-Header_2x25_P2.54mm_Vertical_SMD, F.Cu at (201.2, 27.8)
- added J2: Conn_01x04_Pin, Connector_JST:JST_EH_B4B-EH-A_1x04_P2.50mm_Vertical, F.Cu at (-198.1, 108.6)
- added J3: Conn_01x03_Pin, Connector_JST:JST_EH_B3B-EH-A_1x03_P2.50mm_Vertical, F.Cu at (-135.6, 49.1)
- added J8: Conn_02x25_Odd_Even, Connector_IDC:IDC-Header_2x25_P2.54mm_Vertical_SMD, F.Cu at (200.9, 63.8)
- added J9: Conn_02x25_Odd_Even, Connector_IDC:IDC-Header_2x25_P2.54mm_Vertical_SMD, F.Cu at (114.2, 27.8)
- added R16: 10k, Resistor_SMD:R_0402_1005Metric, F.Cu at (-126.5, 102.2)
- added R17: 4k7, Resistor_SMD:R_0402_1005Metric, F.Cu at (-126.5, 104.2)
- added R19: 4k7, Resistor_SMD:R_0402_1005Metric, F.Cu at (-123.6, 90.3)
- added R20: 10k, Resistor_SMD:R_0402_1005Metric, F.Cu at (-123.6, 92.3)
- added R21: 4k7, Resistor_SMD:R_0402_1005Metric, F.Cu at (-123.6, 94.3)
- added R22: 10k, Resistor_SMD:R_0402_1005Metric, F.Cu at (-123.6, 96.3)
- added R23: 4k7, Resistor_SMD:R_0402_1005Metric, F.Cu at (-123.6, 98.2)
- added R24: 10k, Resistor_SMD:R_0402_1005Metric, F.Cu at (-123.6, 100.2)
- added R25: 10k, Resistor_SMD:R_0402_1005Metric, F.Cu at (-123.6, 102.2)
- added R26: 10k, Resistor_SMD:R_0402_1005Metric, F.Cu at (-123.6, 104.2)
- added R27: 10k, Resistor_SMD:R_0402_1005Metric, F.Cu at (-123.6, 106.2)
- added R29: 10k, Resistor_SMD:R_0402_1005Metric, F.Cu at (-120.7, 92.3)
- added R30: 10k, Resistor_SMD:R_0402_1005Metric, F.Cu at (-120.7, 94.3)
- added R31: 10k, Resistor_SMD:R_0402_1005Metric, F.Cu at (-120.7, 96.3)
- added R32: 10k, Resistor_SMD:R_0402_1005Metric, F.Cu at (-120.7, 98.2)
- added R33: 10k, Resistor_SMD:R_0402_1005Metric, F.Cu at (-120.7, 100.2)
- added R34: 10k, Resistor_SMD:R_0402_1005Metric, F.Cu at (-120.7, 102.2)
- added R35: 10k, Resistor_SMD:R_0402_1005Metric, F.Cu at (-120.7, 104.2)
- added R36: 10k, Resistor_SMD:R_0402_1005Metric, F.Cu at (-120.7, 106.2)
- added R37: 10k, Resistor_SMD:R_0402_1005Metric, F.Cu at (-117.8, 90.3)
- added R38: 10k, Resistor_SMD:R_0402_1005Metric, F.Cu at (-117.8, 92.3)
- added R39: 10k, Resistor_SMD:R_0402_1005Metric, F.Cu at (-117.8, 94.3)
- added R40: 10k, Resistor_SMD:R_0402_1005Metric, F.Cu at (-117.8, 96.3)
- added R41: 10k, Resistor_SMD:R_0402_1005Metric, F.Cu at (-117.8, 98.2)
- added R42: 10k, Resistor_SMD:R_0402_1005Metric, F.Cu at (-117.8, 100.2)
- added R43: 10k, Resistor_SMD:R_0402_1005Metric, F.Cu at (-117.8, 102.2)
- added R44: 10k, Resistor_SMD:R_0402_1005Metric, F.Cu at (-117.8, 104.2)
- added U15: 74CBT16210CDGG, Package_SO:TSSOP-48_6.1x12.5mm_P0.5mm, F.Cu at (196.2, 84.9)
- added U18: 74CBT16210CDGG, Package_SO:TSSOP-48_6.1x12.5mm_P0.5mm, F.Cu at (222.0, 85.2)
- added U19: 74CBT16210CDGG, Package_SO:TSSOP-48_6.1x12.5mm_P0.5mm, F.Cu at (89.0, 47.2)
- added U20: 74CBT16210CDGG, Package_SO:TSSOP-48_6.1x12.5mm_P0.5mm, F.Cu at (117.2, 47.1)
- added U21: 74CBT16210CDGG, Package_SO:TSSOP-48_6.1x12.5mm_P0.5mm, F.Cu at (157.8, 47.2)
- added U22: 74CBT16210CDGG, Package_SO:TSSOP-48_6.1x12.5mm_P0.5mm, F.Cu at (196.2, 47.4)
- added U23: 74CBT16210CDGG, Package_SO:TSSOP-48_6.1x12.5mm_P0.5mm, F.Cu at (221.1, 47.5)
- J5: value Conn_02x25_Odd_Even -> Conn_01x02_Pin; footprint Connector_IDC:IDC-Header_2x25_P2.54mm_Vertical_SMD -> Connector_PinSocket_2.54mm:PinSocket_1x01_P2.54mm_Vertical
- moved V_2 335.7 mm to (-213.1, 101.2)
- moved V_3 335.7 mm to (-208.5, 101.2)
- moved V_4 335.7 mm to (-203.9, 101.2)
- moved Y1 330.8 mm to (-183.7, 108.8)
- moved Y2 318.6 mm to (-178.8, 108.5)
- moved C17 288.4 mm to (-147.4, 42.2)
- moved C20 288.4 mm to (-147.4, 44.7)
- moved C28 288.4 mm to (-147.4, 47.2)
- moved C46 288.4 mm to (-147.4, 49.7)
- moved C47 288.4 mm to (-147.4, 52.2)
- moved FB2 288.4 mm to (-147.4, 54.7)
- moved V_1 284.3 mm to (-134.8, -26.2)
- moved SW1 282.5 mm to (-147.5, 28.3)
- moved SW2 282.5 mm to (-147.5, 33.3)
- moved SW3 282.5 mm to (-147.5, 38.4)
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Connections:
- 23A1024/23LC1 pad 8: VCC -> VCC_5V
- C16 pad 2: VCC -> VCC_5V
- C17 pad 1: VCC -> VCC_5V
- C18 pad 1: VCC -> VCC_5V
- C19 pad 1: VCC -> VCC_5V
- C20 pad 2: VCC -> VCC_5V
- C21 pad 1: VCC -> VCC_5V
- C48 pad 2: VCC -> VCC_5V
- C61 pad 1: Net-(U12-VI) -> VCC_5V
- J4 pad 50: VCC_3 -> Net-(J4-Pin_50)
- J5 pad 1: unconnected-(J5-Pin_1-Pad1) -> /SRAM_CS
- R10 pad 1: VCC -> VCC_5V
- R11 pad 2: unconnected-(R11-Pad2) -> VCC_5V
- R18 pad 2: VCC -> VCC_5V
- U1 pad 1: unconnected-(U1-VCCA-Pad1) -> VCC
- U1 pad 10: unconnected-(U1-GND-Pad10) -> GND
- U1 pad 11: unconnected-(U1-~{OE}-Pad11) -> Net-(U1-~{OE})
- U1 pad 20: unconnected-(U1-VCCB-Pad20) -> VCC_5V
- U10 pad 1: unconnected-(U10-VCCA-Pad1) -> VCC
- U10 pad 10: unconnected-(U10-GND-Pad10) -> GND
- U10 pad 11: unconnected-(U10-~{OE}-Pad11) -> Net-(U10-~{OE})
- U10 pad 20: unconnected-(U10-VCCB-Pad20) -> VCC_5V
- U11 pad 1: unconnected-(U11-VCCA-Pad1) -> VCC
- U11 pad 10: unconnected-(U11-GND-Pad10) -> GND
- U11 pad 11: unconnected-(U11-~{OE}-Pad11) -> Net-(U11-~{OE})
- U11 pad 20: unconnected-(U11-VCCB-Pad20) -> VCC_5V
- U12 pad 3: Net-(U12-VI) -> VCC_5V
- U13 pad 1: unconnected-(U13-VCCA-Pad1) -> VCC
- U13 pad 10: unconnected-(U13-GND-Pad10) -> GND
- U13 pad 11: unconnected-(U13-~{OE}-Pad11) -> Net-(U13-~{OE})
- U13 pad 20: unconnected-(U13-VCCB-Pad20) -> VCC_5V
- U14 pad 15: unconnected-(U14-VCC-Pad15) -> VCC_5V
- U14 pad 17: Net-(U14-GND-Pad17) -> GND
- U14 pad 32: Net-(U14-GND-Pad17) -> GND
- U14 pad 41: Net-(U14-GND-Pad17) -> GND
- U14 pad 47: unconnected-(U14-2~{OE}-Pad47) -> /BUS_1
- U14 pad 48: unconnected-(U14-1~{OE}-Pad48) -> /BUS_1
- U14 pad 8: Net-(U14-GND-Pad17) -> GND
- U16 pad 15: unconnected-(U16-VCC-Pad15) -> VCC_5V
- U16 pad 17: Net-(U16-GND-Pad17) -> GND
- U16 pad 32: Net-(U16-GND-Pad17) -> GND
- U16 pad 41: Net-(U16-GND-Pad17) -> GND
- U16 pad 47: unconnected-(U16-2~{OE}-Pad47) -> /BUS_1
- U16 pad 48: unconnected-(U16-1~{OE}-Pad48) -> /BUS_1
- U16 pad 8: Net-(U16-GND-Pad17) -> GND
- U17 pad 13: unconnected-(U17-2A1-Pad13) -> /burst_1_5V
- U17 pad 14: unconnected-(U17-2A2-Pad14) -> /burst_2_5V
- U17 pad 15: unconnected-(U17-VCC-Pad15) -> VCC_5V
- U17 pad 16: unconnected-(U17-2A3-Pad16) -> /burst_3_5V
- U17 pad 17: Net-(U17-GND-Pad17) -> GND
- U17 pad 18: unconnected-(U17-2A4-Pad18) -> /burst_4_5V
- U17 pad 19: unconnected-(U17-2A5-Pad19) -> /burst_5_5V
- U17 pad 20: unconnected-(U17-2A6-Pad20) -> /burst_6_5V
- U17 pad 21: unconnected-(U17-2A7-Pad21) -> /burst_7_5V
- U17 pad 22: unconnected-(U17-2A8-Pad22) -> /burst_8_5V
- U17 pad 23: unconnected-(U17-2A9-Pad23) -> /burst_9_5V
- U17 pad 24: unconnected-(U17-2A10-Pad24) -> /burst_10_5V
- U17 pad 25: unconnected-(U17-2B10-Pad25) -> /BURST_10.2
- U17 pad 26: unconnected-(U17-2B9-Pad26) -> /BURST_9.2
- U17 pad 27: unconnected-(U17-2B8-Pad27) -> /BURST_8.2
- U17 pad 28: unconnected-(U17-2B7-Pad28) -> /BURST_7.2
- U17 pad 29: unconnected-(U17-2B6-Pad29) -> /BURST_6.2
- U17 pad 30: unconnected-(U17-2B5-Pad30) -> /BURST_5.2
- U17 pad 31: unconnected-(U17-2B4-Pad31) -> /BURST_4.2
- U17 pad 32: Net-(U17-GND-Pad17) -> GND
- U17 pad 33: unconnected-(U17-2B3-Pad33) -> /BURST_3.2
- U17 pad 34: unconnected-(U17-2B2-Pad34) -> /BURST_2.2
- U17 pad 35: unconnected-(U17-2B1-Pad35) -> /BURST_1.2
- U17 pad 41: Net-(U17-GND-Pad17) -> GND
- U17 pad 47: unconnected-(U17-2~{OE}-Pad47) -> /BUS_2
- U17 pad 48: unconnected-(U17-1~{OE}-Pad48) -> /BUS_1
- U17 pad 8: Net-(U17-GND-Pad17) -> GND
- U5 pad 1: unconnected-(U5-VCCA-Pad1) -> VCC
- U5 pad 10: unconnected-(U5-GND-Pad10) -> GND
- U5 pad 11: unconnected-(U5-~{OE}-Pad11) -> Net-(U5-~{OE})
- U5 pad 12: unconnected-(U5-B7-Pad12) -> /INT_5V
- U5 pad 13: unconnected-(U5-B6-Pad13) -> /CTS_5V
- U5 pad 14: unconnected-(U5-B5-Pad14) -> /RTS_5V
- U5 pad 15: unconnected-(U5-B4-Pad15) -> /RAM_CS
- U5 pad 16: unconnected-(U5-B3-Pad16) -> /AT_CS
- U5 pad 17: unconnected-(U5-B2-Pad17) -> /AT_MOSI
- U5 pad 18: unconnected-(U5-B1-Pad18) -> /AT_MISO
- U5 pad 19: unconnected-(U5-B0-Pad19) -> /AT_SCK
- U5 pad 2: unconnected-(U5-A0-Pad2) -> /SCK
- U5 pad 20: unconnected-(U5-VCCB-Pad20) -> VCC_5V
- U5 pad 3: unconnected-(U5-A1-Pad3) -> /MISO
- U5 pad 4: unconnected-(U5-A2-Pad4) -> /MOSI
- U5 pad 5: unconnected-(U5-A3-Pad5) -> /CS
- U5 pad 6: unconnected-(U5-A4-Pad6) -> /SRAM_CS_
- U5 pad 7: unconnected-(U5-A5-Pad7) -> /RTS
- U5 pad 8: unconnected-(U5-A6-Pad8) -> /CTS
- U5 pad 9: unconnected-(U5-A7-Pad9) -> /INT
- U6 pad 25: unconnected-(U6-PA2-Pad25) -> /RTS
- U6 pad 26: unconnected-(U6-PA3-Pad26) -> /CTS
- U6 pad 35: unconnected-(U6-PB0-Pad35) -> /BUS_1_DETECT
- U6 pad 36: unconnected-(U6-PB1-Pad36) -> /BUS_2_DETECT
- U6 pad 37: unconnected-(U6-PB2-Pad37) -> /BUS_3_DETECT
- U6 pad 52: unconnected-(U6-PB13-Pad52) -> /BUS_4_DETECT
- U6 pad 53: unconnected-(U6-PB14-Pad53) -> /INT
- U6 pad 71: unconnected-(U6-PA12-Pad71) -> /SRAM_CS
- U7 pad 18: VCC -> VCC_5V
- U7 pad 2: unconnected-(U7-PD4-Pad2) -> /RTS_5V
- U7 pad 21: Net-(U7-GND-Pad21) -> GND
- U7 pad 3: Net-(U7-GND-Pad21) -> GND
- U7 pad 32: unconnected-(U7-PD2-Pad32) -> /INT_5V
- U7 pad 5: Net-(U7-GND-Pad21) -> GND
- U7 pad 9: unconnected-(U7-PD5-Pad9) -> /CTS_5V
- U8 pad 1: unconnected-(U8-VCCA-Pad1) -> VCC
- U8 pad 10: unconnected-(U8-GND-Pad10) -> GND
- U8 pad 11: unconnected-(U8-~{OE}-Pad11) -> Net-(U8-~{OE})
- U8 pad 20: unconnected-(U8-VCCB-Pad20) -> VCC_5V
- U9 pad 1: unconnected-(U9-VCCA-Pad1) -> VCC
- U9 pad 10: unconnected-(U9-GND-Pad10) -> GND
- U9 pad 11: unconnected-(U9-~{OE}-Pad11) -> Net-(U9-~{OE})
- U9 pad 20: unconnected-(U9-VCCB-Pad20) -> VCC_5V
Routing:
- net /burst_17_5V: track 0.00 -> 229.5 mm, vias 0 -> 3
- net /burst_18_5V: track 0.00 -> 228.9 mm, vias 0 -> 3
- net /burst_19_5V: track 0.00 -> 227.9 mm, vias 0 -> 3
- net /burst_33_5V: track 0.00 -> 226.2 mm, vias 0 -> 3
- net /burst_20_5V: track 0.00 -> 225.5 mm, vias 0 -> 3
- net /burst_34_5V: track 0.00 -> 223.5 mm, vias 0 -> 3
- net /burst_35_5V: track 0.00 -> 222.1 mm, vias 0 -> 3
- net /burst_11_5V: track 0.00 -> 221.0 mm, vias 0 -> 3
- net /burst_12_5V: track 0.00 -> 221.0 mm, vias 0 -> 3
- net /burst_36_5V: track 0.00 -> 220.9 mm, vias 0 -> 3
- net /burst_37_5V: track 0.00 -> 220.5 mm, vias 0 -> 3
- net /burst_13_5V: track 0.00 -> 220.1 mm, vias 0 -> 3
- net /burst_14_5V: track 0.00 -> 220.0 mm, vias 0 -> 3
- net /burst_38_5V: track 0.00 -> 219.5 mm, vias 0 -> 3
- net /burst_15_5V: track 0.00 -> 219.0 mm, vias 0 -> 3
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Other:
- board outline added: 187 x 162 mm
- copper layers 2 -> 4

Commit message: .
Parts:
- removed R26, R27, R30, R31, R33, R34, R36, R37: 10k, Resistor_SMD:R_0402_1005Metric
- moved Y1 369.7 mm to (185.2, 133.6)
- moved R16 368.2 mm to (238.5, 53.6)
- moved R23 364.6 mm to (235.4, 34.9), turned to 90 degrees
- moved R17 364.4 mm to (234.3, 53.6), turned to 180 degrees
- moved R24 364.2 mm to (235.4, 38.7), turned to -90 degrees
- moved C28 330.4 mm to (174.4, 121.8)
- moved C12 324.8 mm to (185.1, 137.0)
- moved C1 323.6 mm to (175.7, 143.8), turned to 180 degrees
- moved C15 322.3 mm to (185.1, 130.2), turned to 180 degrees
- moved C10 321.4 mm to (179.9, 137.8)
- moved C5 321.0 mm to (178.8, 135.5), turned to -90 degrees
- moved C6 320.2 mm to (174.9, 146.2)
- moved C9 319.9 mm to (174.9, 145.0)
- moved C13 317.0 mm to (179.6, 130.7), turned to -90 degrees
- moved C3 314.5 mm to (174.3, 124.2)
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Connections:
- U6 pad 1: /burst_19 -> unconnected-(U6-PE2-Pad1)
- U6 pad 15: /burst_1 -> unconnected-(U6-PC0-Pad15)
- U6 pad 16: /burst_2 -> unconnected-(U6-PC1-Pad16)
- U6 pad 17: /burst_3 -> unconnected-(U6-PC2-Pad17)
- U6 pad 18: /burst_4 -> unconnected-(U6-PC3-Pad18)
- U6 pad 2: /burst_20 -> unconnected-(U6-PE3-Pad2)
- U6 pad 25: /RTS -> /burst_40
- U6 pad 26: /CTS -> /burst_39
- U6 pad 3: /burst_21 -> unconnected-(U6-PE4-Pad3)
- U6 pad 33: /burst_5 -> /burst_38
- U6 pad 34: /burst_6 -> /burst_37
- U6 pad 35: /BUS_1_DETECT -> /burst_36
- U6 pad 36: /BUS_2_DETECT -> /burst_35
- U6 pad 37: /BUS_3_DETECT -> /burst_34
- U6 pad 38: /burst_24 -> /burst_33
- U6 pad 39: /burst_25 -> /burst_32
- U6 pad 4: /burst_22 -> unconnected-(U6-PE5-Pad4)
- U6 pad 40: /burst_26 -> /burst_31
- U6 pad 41: /burst_27 -> /burst_30
- U6 pad 42: /burst_28 -> /burst_29
- U6 pad 43: /burst_29 -> /burst_28
- U6 pad 44: /burst_30 -> /burst_27
- U6 pad 45: /burst_31 -> /burst_26
- U6 pad 46: /burst_32 -> /burst_25
- U6 pad 5: /burst_23 -> unconnected-(U6-PE6-Pad5)
- U6 pad 51: /J_C -> /burst_24
- U6 pad 52: /BUS_4_DETECT -> /burst_23
- U6 pad 53: /INT -> /burst_22
- U6 pad 54: /burst_17 -> /burst_21
- U6 pad 55: /burst_41 -> /burst_20
- U6 pad 56: /burst_42 -> /burst_19
- U6 pad 57: /burst_43 -> /burst_18
- U6 pad 58: /burst_44 -> /burst_17
- U6 pad 59: /burst_45 -> /burst_16
- U6 pad 60: /burst_46 -> /burst_15
- U6 pad 61: /burst_47 -> /burst_14
- U6 pad 62: /burst_48 -> /burst_13
- U6 pad 63: /burst_7 -> /burst_12
- U6 pad 64: /burst_8 -> /burst_11
- U6 pad 65: /burst_9 -> /burst_10
- U6 pad 66: /burst_10 -> /burst_9
- U6 pad 67: /BUS_1 -> /burst_8
- U6 pad 68: /BUS_2 -> /burst_7
- U6 pad 69: /BUS_3 -> /burst_6
- U6 pad 7: /burst_14 -> unconnected-(U6-PC13-Pad7)
- U6 pad 70: /BUS_4 -> /burst_5
- U6 pad 71: /SRAM_CS -> /burst_4
- U6 pad 78: /burst_11 -> /burst_3
- U6 pad 79: /burst_12 -> /burst_2
- U6 pad 8: /burst_15 -> unconnected-(U6-PC14-Pad8)
- U6 pad 80: /burst_13 -> /burst_1
- U6 pad 81: /burst_33 -> /burst_41
- U6 pad 82: /burst_34 -> /burst_42
- U6 pad 83: /burst_35 -> /burst_43
- U6 pad 84: /burst_36 -> /burst_44
- U6 pad 85: /burst_37 -> /burst_45
- U6 pad 86: /burst_38 -> /burst_46
- U6 pad 87: /burst_39 -> /burst_47
- U6 pad 88: /burst_40 -> /burst_48
- U6 pad 9: /burst_16 -> unconnected-(U6-PC15-Pad9)
- U6 pad 97: /burst_18 -> unconnected-(U6-PE0-Pad97)
Routing:
- net /burst_1_5V: track 133.2 -> 255.9 mm, vias 4 -> 6
- net /burst_2_5V: track 132.8 -> 253.8 mm, vias 4 -> 6
- net /burst_3_5V: track 132.5 -> 249.9 mm, vias 4 -> 6
- net /burst_4_5V: track 121.2 -> 235.6 mm, vias 4 -> 6
- net /burst_5_5V: track 120.6 -> 232.4 mm, vias 4 -> 6
- net /burst_6_5V: track 120.4 -> 229.3 mm, vias 4 -> 6
- net /burst_7_5V: track 120.1 -> 226.7 mm, vias 4 -> 6
- net /burst_8_5V: track 119.7 -> 218.3 mm, vias 4 -> 6
- net /burst_9_5V: track 133.7 -> 228.3 mm, vias 4 -> 6
- net /burst_10_5V: track 133.0 -> 222.5 mm, vias 4 -> 6
- net /burst_1: track 0.00 -> 82.3 mm
- net /burst_2: track 0.00 -> 80.5 mm
- net /burst_3: track 0.00 -> 78.9 mm
- net /burst_4: track 0.00 -> 66.4 mm
- net /burst_5: track 0.00 -> 65.6 mm
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
Commit message: .
Parts:
- removed C1_Crystal1, C2_Crystal1: C_Small, Capacitor_THT:CP_Radial_D5.0mm_P2.50mm
- added 220UF1: C_Polarized, Capacitor_THT:C_Disc_D3.0mm_W1.6mm_P2.50mm, F.Cu at (246.3, 140.1)
- added 220UF2: C_Polarized, Capacitor_THT:C_Disc_D3.0mm_W1.6mm_P2.50mm, F.Cu at (246.3, 143.3)
- added C22: 10p, Capacitor_SMD:C_0402_1005Metric, F.Cu at (95.3, 110.9)
- added C23: 10p, Capacitor_SMD:C_0402_1005Metric, F.Cu at (90.3, 110.9)
- added C24: 100n, Capacitor_SMD:C_0402_1005Metric, F.Cu at (130.8, 109.2)
- added C25: 100n, Capacitor_SMD:C_0402_1005Metric, F.Cu at (111.3, 108.8)
- added C26: 100n, Capacitor_SMD:C_0402_1005Metric, F.Cu at (148.5, 110.5)
- added C27: 100n, Capacitor_SMD:C_0402_1005Metric, F.Cu at (165.3, 110.5)
- added C29: 100n, Capacitor_SMD:C_0402_1005Metric, F.Cu at (184.3, 110.8)
- added C30: 100n, Capacitor_SMD:C_0402_1005Metric, F.Cu at (202.0, 110.8)
- added C31: 2.2u, Capacitor_SMD:C_0402_1005Metric, F.Cu at (191.8, 114.2)
- added C32: 100n, Capacitor_SMD:C_0402_1005Metric, F.Cu at (193.0, 114.0)
- added C33: 2.2u, Capacitor_SMD:C_0402_1005Metric, F.Cu at (192.8, 111.2)
- added C34: 100n, Capacitor_SMD:C_0402_1005Metric, F.Cu at (191.5, 111.2)
- added C35: 2.2u, Capacitor_SMD:C_0402_1005Metric, F.Cu at (173.8, 111.0)
- added C36: 100n, Capacitor_SMD:C_0402_1005Metric, F.Cu at (175.0, 111.0)
- added C37: 2.2u, Capacitor_SMD:C_0402_1005Metric, F.Cu at (173.8, 113.3)
- added C38: 100n, Capacitor_SMD:C_0402_1005Metric, F.Cu at (175.0, 113.3)
- added C39: 2.2u, Capacitor_SMD:C_0402_1005Metric, F.Cu at (155.0, 111.0)
- added C41: 100n, Capacitor_SMD:C_0402_1005Metric, F.Cu at (156.2, 111.0)
- added C42: 2.2u, Capacitor_SMD:C_0402_1005Metric, F.Cu at (155.2, 113.8)
- added C43: 100n, Capacitor_SMD:C_0402_1005Metric, F.Cu at (122.0, 113.3)
- added C45: 2.2u, Capacitor_SMD:C_0402_1005Metric, F.Cu at (138.0, 110.2)
- added C49: 100n, Capacitor_SMD:C_0402_1005Metric, F.Cu at (122.0, 109.7)
- added C50: 2.2u, Capacitor_SMD:C_0402_1005Metric, F.Cu at (100.5, 114.3)
- added C51: 100n, Capacitor_SMD:C_0402_1005Metric, F.Cu at (102.0, 114.0)
- added C52: 2.2u, Capacitor_SMD:C_0402_1005Metric, F.Cu at (100.5, 110.2)
- added C53: 100n, Capacitor_SMD:C_0402_1005Metric, F.Cu at (102.0, 110.2)
- added C54: 2.2u, Capacitor_SMD:C_0402_1005Metric, F.Cu at (138.0, 113.3)
- added C55: 100n, Capacitor_SMD:C_0402_1005Metric, F.Cu at (156.5, 113.8)
- added C56: 2.2u, Capacitor_SMD:C_0402_1005Metric, F.Cu at (120.5, 109.5)
- added C57: 100n, Capacitor_SMD:C_0402_1005Metric, F.Cu at (139.2, 110.2)
- added C58: 2.2u, Capacitor_SMD:C_0402_1005Metric, F.Cu at (120.8, 113.3)
- added C59: 100n, Capacitor_SMD:C_0402_1005Metric, F.Cu at (139.2, 113.2)
- added C60: 47pf, Capacitor_SMD:C_0402_1005Metric, F.Cu at (122.0, 143.8)
- added C63: 47pf, Capacitor_SMD:C_0402_1005Metric, F.Cu at (125.5, 143.7)
- added C64: 100n, Capacitor_SMD:C_0402_1005Metric, F.Cu at (142.5, 153.5)
- added C65: 4.7u, Capacitor_SMD:C_0603_1608Metric, F.Cu at (144.7, 154.5)
- added C66: 100n, Capacitor_SMD:C_0402_1005Metric, F.Cu at (147.8, 139.5)
- added C67: 100n, Capacitor_SMD:C_0402_1005Metric, F.Cu at (144.8, 152.5)
- added D1: LED, LED_SMD:LED_0603_1608Metric, F.Cu at (152.5, 154.0)
- added D2: LED, LED_SMD:LED_0603_1608Metric, F.Cu at (164.2, 154.0)
- added D7: LED, LED_SMD:LED_0603_1608Metric, F.Cu at (158.5, 154.0)
- added J15: PJ-102A, Connector_BarrelJack:BarrelJack_Horizontal, F.Cu at (107.8, 148.0)
- added J6: USB_A, Connector_USB:USB_B_Lumberg_2411_02_Horizontal, F.Cu at (127.2, 147.0)
- added R26: 4k7, Resistor_SMD:R_0402_1005Metric, F.Cu at (138.2, 149.0)
- added R27: 10k, Resistor_SMD:R_0402_1005Metric, F.Cu at (138.8, 151.3)
- added R30: 200, Resistor_SMD:R_0402_1005Metric, F.Cu at (154.5, 154.0)
- added R31: 200, Resistor_SMD:R_0402_1005Metric, F.Cu at (160.5, 154.2)
- added R33: 10k, Resistor_SMD:R_0402_1005Metric, F.Cu at (141.5, 140.2)
- added R34: 200, Resistor_SMD:R_0402_1005Metric, F.Cu at (166.2, 154.2)
- added SW5: SW_Push, Button_Switch_THT:SW_PUSH_1P1T_6x3.5mm_H4.3_APEM_MJTP1243, F.Cu at (187.8, 152.8)
- added U3: FT232RL, Package_SO:SSOP-28_5.3x10.2mm_P0.65mm, F.Cu at (146.3, 146.2)
- moved SW2 373.4 mm to (213.0, 152.8)
- moved SW3 360.1 mm to (200.5, 152.8)
- moved R28 352.4 mm to (184.5, 155.0)
- moved SW1 338.1 mm to (175.5, 152.8)
- moved J1 313.1 mm to (234.2, 135.5), turned to 90 degrees
- moved J3 306.0 mm to (234.5, 121.8), turned to 90 degrees
- moved J2 286.6 mm to (235.0, 101.0), turned to -90 degrees
- moved C21 246.1 mm to (97.2, 129.8)
- moved C18 243.8 mm to (94.2, 130.5), turned to -90 degrees
- moved C48 242.9 mm to (101.0, 145.1), turned to -90 degrees
- moved C62 232.2 mm to (88.5, 154.2), turned to 180 degrees
- moved C61 231.0 mm to (91.8, 137.5)
- moved C17 227.7 mm to (92.2, 130.8), turned to -90 degrees
- moved J5 225.1 mm to (78.6, 164.0)
- moved C14 211.1 mm to (45.1, 183.1)
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Connections:
- J12 pad 1: /MOSI -> /AT_MOSI
- J12 pad 5: /CS -> /AT_CS
- J12 pad 7: /SCK -> /AT_SCK
- J12 pad 9: /MISO -> /AT_MISO
- U7 pad 20: VCC -> VCC_5V
Routing:
- net VCC_5V: track 0.00 -> 683.3 mm, vias 0 -> 17
- net GND: track 34.6 -> 247.1 mm, vias 0 -> 84
- net /NRST: track 0.00 -> 70.8 mm, vias 0 -> 1
- net Net-(U3-~{RESET}): track 0.00 -> 68.3 mm, vias 0 -> 1
- net /JTMS-SWDIO: track 0.00 -> 60.6 mm, vias 0 -> 4
- net /JTCK-SWCLK: track 0.00 -> 54.3 mm, vias 0 -> 3
- net /TRACESWO - JTDO: track 0.00 -> 51.3 mm
- net /D+: track 0.00 -> 49.7 mm
- net VCC: track 21.1 -> 70.8 mm, vias 0 -> 18
- net /JTDI: track 0.00 -> 47.8 mm, vias 0 -> 3
- net /D-: track 0.00 -> 47.5 mm
- net /NJRST: track 0.00 -> 37.6 mm
- net Net-(U6-BOOT0): track 0.00 -> 26.9 mm, vias 0 -> 1
- net /AT_SCK: track 0.00 -> 19.3 mm, vias 0 -> 1
- net Net-(D1-K): track 0.00 -> 17.8 mm, vias 0 -> 2
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- added copper zone on F.Cu, net GND
- added copper zone on In2.Cu, net GND
- added copper zone on B.Cu, net VCC
- added copper zone on F.Cu, net VCC
- added copper zone on F.Cu, net VCC_5V
Other:
- board size 187 x 162 mm -> 163.4 x 136.9 mm

Commit message: .
Parts:
- added ? (x2): , , F.Cu at (105.7, 111.7)
- added C4321: 16PK4700MEFC12.5X25, Capacitor_THT:CP_Radial_D5.0mm_P2.50mm, F.Cu at (106.5, 130.8)
- added C4322: T520Y337M006ATE040, Capacitor_SMD:CP_Elec_10x10, F.Cu at (131.8, 130.0)
- added SPEAKER1: Conn_01x03_Pin, Connector_JST:JST_EH_B3B-EH-A_1x03_P2.50mm_Vertical, F.Cu at (236.8, 111.0)
- J5: footprint Connector_PinSocket_2.54mm:PinSocket_1x01_P2.54mm_Vertical -> Connector_PinSocket_2.54mm:PinSocket_1x02_P2.54mm_Vertical
- V_1, V_2, V_3, V_4: footprint Connector_PinHeader_2.54mm:PinHeader_1x02_P2.54mm_Vertical -> Connector_JST:JST_EH_B2B-EH-A_1x02_P2.50mm_Vertical
- moved V_1 326.4 mm to (237.0, 151.0), turned to -90 degrees
- moved V_2 318.2 mm to (237.0, 141.8), turned to -90 degrees
- moved V_3 306.1 mm to (236.8, 123.0), turned to -90 degrees
- moved V_4 305.7 mm to (236.8, 132.5), turned to -90 degrees
- moved R15 276.9 mm to (232.5, 127.2)
- moved R8 268.1 mm to (231.3, 101.2), turned to 180 degrees
- moved R3 214.9 mm to (231.2, 84.2), turned to 180 degrees
- moved R4 214.7 mm to (231.2, 86.8), turned to 180 degrees
- moved R5 214.5 mm to (231.2, 89.2), turned to 180 degrees
- moved R6 214.4 mm to (231.2, 91.8), turned to 180 degrees
- moved R7 212.9 mm to (231.2, 98.8), turned to 180 degrees
- moved R9 206.2 mm to (231.2, 103.8), turned to 180 degrees
- moved R14 202.8 mm to (232.0, 137.0)
- moved R13 202.6 mm to (232.7, 145.8)
- moved R12 201.9 mm to (232.5, 155.2)
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Connections:
- JTAG1 pad 1: 3.3V -> VCC
- JTAG1 pad 2: 3.3V -> VCC
- Q1 pad 3: unconnected-(Q1-D-Pad3) -> VCC_5V
- Q2 pad 3: unconnected-(Q2-D-Pad3) -> VCC_5V
- Q3 pad 3: unconnected-(Q3-D-Pad3) -> VCC_5V
- Q4 pad 3: unconnected-(Q4-D-Pad3) -> VCC_5V
- U3 pad 1: /TXD_CONV -> /RX
- U3 pad 5: /RXD_CONV -> /TX
- U6 pad 1: unconnected-(U6-PE2-Pad1) -> /BUS_2
- U6 pad 15: unconnected-(U6-PC0-Pad15) -> /J_UP
- U6 pad 16: unconnected-(U6-PC1-Pad16) -> /J_DOWN
- U6 pad 17: unconnected-(U6-PC2-Pad17) -> /J_LEFT
- U6 pad 18: unconnected-(U6-PC3-Pad18) -> /J_RIGHT
- U6 pad 2: unconnected-(U6-PE3-Pad2) -> /BUS_3
- U6 pad 3: unconnected-(U6-PE4-Pad3) -> /BUS_4
- U6 pad 4: unconnected-(U6-PE5-Pad4) -> /BUS_1_DETECT
- U6 pad 47: /J_B -> /BUS_4_DETECT
- U6 pad 5: unconnected-(U6-PE6-Pad5) -> /BUS_2_DETECT
- U6 pad 7: unconnected-(U6-PC13-Pad7) -> /J_C
- U6 pad 8: unconnected-(U6-PC14-Pad8) -> /J_A
- U6 pad 9: unconnected-(U6-PC15-Pad9) -> /J_B
- U6 pad 91: /J_UP -> /RTS
- U6 pad 92: /J_DOWN -> /CTS
- U6 pad 93: /J_LEFT -> /SRAM_CS
- U6 pad 95: /J_RIGHT -> /INT
- U6 pad 96: /J_A -> /BUS_3_DETECT
- U6 pad 97: unconnected-(U6-PE0-Pad97) -> /BUS_1
- U7 pad 4: Net-(U7-VCC-Pad4) -> VCC_5V
- U7 pad 6: Net-(U7-VCC-Pad4) -> VCC_5V
Routing:
- net VCC_5V: track 683.3 -> 882.1 mm, vias 17 -> 28
- net /V_1: track 0.00 -> 158.7 mm, vias 0 -> 6
- net /V_2: track 0.00 -> 153.9 mm, vias 0 -> 8
- net /SPEAKER_R: track 0.00 -> 151.8 mm, vias 0 -> 8
- net /SPEAKER_L: track 0.00 -> 146.6 mm, vias 0 -> 10
- net /V_4: track 0.00 -> 145.2 mm, vias 0 -> 10
- net /V_3: track 0.00 -> 135.3 mm, vias 0 -> 8
- net Net-(U7-~{RESET}/PC6): track 0.00 -> 126.4 mm, vias 0 -> 2
- net /BUS_1: track 0.00 -> 104.6 mm, vias 0 -> 4
- net /J_UP: track 0.00 -> 103.6 mm, vias 0 -> 1
- net /J_DOWN: track 0.00 -> 100.1 mm, vias 0 -> 1
- net VCCA: track 4.25 -> 100.7 mm, vias 0 -> 6
- net /J_LEFT: track 0.00 -> 95.1 mm, vias 0 -> 1
- net /J_C: track 0.00 -> 94.2 mm, vias 0 -> 2
- net /J_RIGHT: track 0.00 -> 88.7 mm, vias 0 -> 1
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Other:
- board text added: "DOWN"
- board text added: "GND"
- board text added: "JA"
- board text added: "JB"
- board text added: "JC"
- board text added: "LEFT"
- board text added: "RIGHT"
- board text added: "RX"
- board text added: "SPEAKER_L"
- board text added: "SPEAKER_R"
- board text added: "TX"
- board text added: "UP"
- board text added: "V1"
- board text added: "V2"
- board text added: "V3"
- board text added: "V4"

Commit message: .
Connections:
- U6 pad 96: /BUS_3_DETECT -> /BUS_1
- U6 pad 97: /BUS_1 -> /BUS_3_DETECT
Routing:
- net /BUS_3_DETECT: track 3.40 -> 206.9 mm, vias 0 -> 4
- net /BUS_3: track 85.7 -> 282.6 mm, vias 0 -> 6
- net /BUS_1_DETECT: track 2.16 -> 163.5 mm, vias 0 -> 6
- net /BUS_1: track 104.6 -> 256.0 mm, vias 4 -> 8
- net /BUS_4_DETECT: track 2.76 -> 147.9 mm, vias 0 -> 4
- net /BUS_4: track 81.5 -> 224.1 mm, vias 0 -> 6
- net /BUS_2_DETECT: track 3.16 -> 132.6 mm, vias 0 -> 4
- net /BUS_2: track 79.7 -> 183.7 mm, vias 4 -> 8
- net VCC: track 100.0 -> 101.5 mm, vias 27 -> 28
