File: stm/ws2812b_module/kicad/kicad.kicad_pcb (KiCad board)
At the start: 4 copper layers, 163.4 x 136.9 mm, 168 parts, among them J1 Conn_01x03_Pin, J10 Conn_02x25_Odd_Even, J12 USB_ASP, J15 PJ-102A, J2 Conn_01x04_Pin, J3 Conn_01x03_Pin, J4 Conn_02x25_Odd_Even, J5 Conn_01x02_Pin, J6 USB_A, J8 Conn_02x25_Odd_Even, J9 Conn_02x25_Odd_Even, Q1 T2N7002AK, Q2 T2N7002AK, Q3 T2N7002AK, Q4 T2N7002AK, SW1 SW_Push, SW2 SW_Push, SW3 SW_Push, SW5 SW_Push, U1 FXMA108, U10 FXMA108, U11 FXMA108, U12 AMS1117-3.3, U13 FXMA108, U14 74CBT16210CDGG, U15 74CBT16210CDGG, U16 74CBT16210CDGG, U17 74CBT16210CDGG, U18 74CBT16210CDGG, U19 74CBT16210CDGG, U20 74CBT16210CDGG, U21 74CBT16210CDGG, U22 74CBT16210CDGG, U23 74CBT16210CDGG, U3 FT232RL, U5 FXMA108, U6 STM32H563VGTx, U7 ATmega328-A, U8 FXMA108, U9 FXMA108, Y1 26MHz, Y2 Crystal

Commit message: .
Parts:
- added ATUART1: Conn_01x03_Pin, Connector_JST:JST_EH_B3B-EH-A_1x03_P2.50mm_Vertical, F.Cu at (84.9, 154.4)
- added LCD1: Conn_01x04_Pin, Connector_JST:JST_EH_B4B-EH-A_1x04_P2.50mm_Vertical, F.Cu at (79.6, 103.5)
- moved C47 2.63 mm to (94.8, 155.5)
- moved C62 2.56 mm to (90.7, 155.5)
- renumbered SW3 to ATRESET1, SW1 to BOOT0, SW5 to FRESET1, D7 to FRX1, D1 to FTX1, J4 to GRID1, J8 to GRID2, J9 to GRID3, J10 to GRID4, D2 to PWR1, SW2 to STRESET1, J1 to STUART1, J12 to USBASP1
Connections:
- net /burst_1 renamed /burst_1_
- net /burst_10 renamed /burst_10_
- net /burst_11 renamed /burst_11_
- net /burst_12 renamed /burst_12_
- net /burst_13 renamed /burst_13_
- net /burst_14 renamed /burst_14_
- net /burst_15 renamed /burst_15_
- net /burst_16 renamed /burst_16_
- net /burst_17 renamed /burst_17_
- net /burst_18 renamed /burst_18_
- net /burst_19 renamed /burst_19_
- net /burst_2 renamed /burst_2_
- net /burst_20 renamed /burst_20_
- net /burst_21 renamed /burst_21_
- net /burst_22 renamed /burst_22_
- net /burst_23 renamed /burst_23_
- net /burst_24 renamed /burst_24_
- net /burst_25 renamed /burst_25_
- net /burst_26 renamed /burst_26_
- net /burst_27 renamed /burst_27_
- net /burst_28 renamed /burst_28_
- net /burst_29 renamed /burst_29_
- net /burst_3 renamed /burst_3_
- net /burst_30 renamed /burst_30_
- net /burst_31 renamed /burst_31_
- net /burst_32 renamed /burst_32_
- net /burst_33 renamed /burst_33_
- net /burst_34 renamed /burst_34_
- net /burst_35 renamed /burst_35_
- net /burst_36 renamed /burst_36_
- net /burst_37 renamed /burst_37_
- net /burst_38 renamed /burst_38_
- net /burst_39 renamed /burst_39_
- net /burst_4 renamed /burst_4_
- net /burst_40 renamed /burst_40_
- net /burst_41 renamed /burst_41_
- net /burst_42 renamed /burst_42_
- net /burst_43 renamed /burst_43_
- net /burst_44 renamed /burst_44_
- net /burst_45 renamed /burst_45_
- net /burst_46 renamed /burst_46_
- net /burst_47 renamed /burst_47_
- net /burst_48 renamed /burst_48_
- net /burst_5 renamed /burst_5_
- net /burst_6 renamed /burst_6_
- net /burst_7 renamed /burst_7_
- net /burst_8 renamed /burst_8_
- net /burst_9 renamed /burst_9_
- 23A1024/23LC1 pad 2: /AT_MOSI -> /AT_MISO
- 23A1024/23LC1 pad 5: /AT_MISO -> /AT_MOSI
- GRID3 pad 30: /BURST_30,3 -> /BURST_30.3
Routing:
- net /AT_TX: track 0.00 -> 52.6 mm, vias 0 -> 1
- net /AT_RX: track 0.00 -> 52.2 mm, vias 0 -> 1
- net /SDA: track 0.00 -> 38.9 mm, vias 0 -> 1
- net /SCL: track 0.00 -> 31.3 mm, vias 0 -> 1
- net /BURST_30.3: track 0.00 -> 21.2 mm
- net VCC_5V: track 882.1 -> 896.0 mm
- net VCC: track 101.5 -> 110.7 mm, vias 28 -> 29
- net /AT_MOSI: track 69.3 -> 74.3 mm
- net GND: track 315.6 -> 320.5 mm, vias 115 -> 103
- net /AT_MISO: track 82.7 -> 78.1 mm
- net /JTMS-SWDIO: track 60.6 -> 61.7 mm
- net /burst_25_5V: track 249.7 -> 250.6 mm
- net /burst_24_5V: track 237.9 -> 238.7 mm
- net /burst_26_5V: track 248.8 -> 249.6 mm
- net /burst_28_5V: track 243.9 -> 244.7 mm
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- added copper zone on B.Cu, net (none)
- added copper zone on In1.Cu, net (none)
- added copper zone on In2.Cu, net (none)
