File: stm/ws2812b_module/kicad/kicad.kicad_sch (KiCad schematic)
At the start: 89 parts, among them J1 Conn_01x03_Pin, J12 USB_ASP, J2 Conn_01x04_Pin, J3 Conn_01x03_Pin, J4 Conn_02x25_Odd_Even, J5 Conn_02x25_Odd_Even, J6 Conn_02x25_Odd_Even, J7 Conn_02x25_Odd_Even, Q1 T2N7002AK, Q2 T2N7002AK, Q3 T2N7002AK, Q4 T2N7002AK, SW1 SW_Push, SW2 SW_Push, SW3 SW_Push, U1 FXMA108, U10 FXMA108, U11 FXMA108, U12 AMS1117-3.3, U13 FXMA108, U14 74CBT16210CDGG, U16 74CBT16210CDGG, U17 74CBT16210CDGG, U2 FXMA108, U3 FXMA108, U4 FXMA108, U5 FXMA108, U6 STM32H563VGTx, U7 ATmega328-A, U8 FXMA108, U9 FXMA108, Y1 26MHz, Y2 Crystal

Commit message: .
Parts:
- removed J5, J6, J7: Conn_02x25_Odd_Even, Connector_IDC:IDC-Header_2x25_P2.54mm_Vertical_SMD, symbol Connector_Generic:Conn_02x25_Odd_Even
- removed U2, U3, U4: FXMA108, Package_DFN_QFN:WQFN-20-1EP_2.5x4.5mm_P0.5mm_EP1x2.9mm, symbol Logic_LevelTranslator:FXMA108
- added J10, J8, J9: Conn_02x25_Odd_Even, Connector_IDC:IDC-Header_2x25_P2.54mm_Vertical_SMD, symbol Connector_Generic:Conn_02x25_Odd_Even
- added J5: Conn_01x02_Pin, Connector_PinSocket_2.54mm:PinSocket_1x01_P2.54mm_Vertical, symbol Connector:Conn_01x02_Pin
- added R16, R20, R22, R24, R25, R26, R27, R29, R30, R31, R32, R33, R34, R35, R36, R37, R38, R39, R40, R41, R42, R43, R44: 10k, Resistor_SMD:R_0402_1005Metric, symbol Device:R
- added R17, R19, R21, R23: 4k7, Resistor_SMD:R_0402_1005Metric, symbol Device:R
- added U15, U18, U19, U20, U21, U22, U23: 74CBT16210CDGG, Package_SO:TSSOP-48_6.1x12.5mm_P0.5mm, symbol 74xx:74CBT16210CDGG
- J1, J3: footprint (none) -> Connector_JST:JST_EH_B3B-EH-A_1x03_P2.50mm_Vertical
- J2: footprint (none) -> Connector_JST:JST_EH_B4B-EH-A_1x04_P2.50mm_Vertical
Connections:
- net AT_CS: now also U5.16 (B3)
- net AT_MISO: now also U5.18 (B1)
- net AT_MOSI: now also U5.17 (B2)
- net AT_SCK: now also U5.19 (B0)
- net BUS_1: now also U14.47 (2~{OE}), U14.48 (1~{OE}), U16.47 (2~{OE}), U16.48 (1~{OE}), U17.48 (1~{OE}), R25.2, R26.2, R27.2
- net BUS_2: now also U17.47 (2~{OE}), R29.2, R30.2, R31.2, U15.47 (2~{OE}), U15.48 (1~{OE}), U18.47 (2~{OE}), U18.48 (1~{OE})
- net BUS_3: now also R32.2, R33.2, R34.2, U19.47 (2~{OE}), U19.48 (1~{OE}), U20.47 (2~{OE}), U20.48 (1~{OE}), U21.48 (1~{OE})
- net BUS_4: now also R35.2, R36.2, R37.2, U21.47 (2~{OE}), U22.47 (2~{OE}), U22.48 (1~{OE}), U23.47 (2~{OE}), U23.48 (1~{OE})
- net CS: now also U5.5 (A3)
- net GND: now also U1.10 (GND), U10.10 (GND), U11.10 (GND), U13.10 (GND), U14.17 (GND), U14.32 (GND), U14.41 (GND), U14.8 (GND), U16.17 (GND), U16.32 (GND), U16.41 (GND), U16.8 (GND), U17.17 (GND), U17.32 (GND), U17.41 (GND), U17.8 (GND), U5.10 (GND), U7.21 (GND), U7.3 (GND), U7.5 (GND), U8.10 (GND), U9.10 (GND), J10.49 (Pin_49), J8.49 (Pin_49), J9.49 (Pin_49), R16.2, R20.2, R22.2, R24.2, R38.2, R39.2, R40.2, R41.2, R42.2, R43.2, R44.2, U15.17 (GND), U15.32 (GND), U15.41 (GND), U15.8 (GND), U18.17 (GND), U18.32 (GND), U18.41 (GND), U18.8 (GND), U19.17 (GND), U19.32 (GND), U19.41 (GND), U19.8 (GND), U20.17 (GND), U20.32 (GND), U20.41 (GND), U20.8 (GND), U21.17 (GND), U21.32 (GND), U21.41 (GND), U21.8 (GND), U22.17 (GND), U22.32 (GND), U22.41 (GND), U22.8 (GND), U23.17 (GND), U23.32 (GND), U23.41 (GND), U23.8 (GND)
- net MISO: now also U5.3 (A1)
- net MOSI: now also U5.4 (A2)
- net RAM_CS: now also U5.15 (B4)
- net SCK: now also U5.2 (A0)
- net VCC: now also U1.1 (VCCA), U10.1 (VCCA), U11.1 (VCCA), U13.1 (VCCA), U5.1 (VCCA), U8.1 (VCCA), U9.1 (VCCA), R25.1, R26.1, R27.1, R29.1, R30.1, R31.1, R32.1, R33.1, R34.1, R35.1, R36.1, R37.1; no longer 23A1024/23LC1.8 (VCC), C16.2, C17.1, C18.1, C19.1, C20.2, C21.1, C48.2, R10.1, R18.2, U7.18 (AVCC)
- net burst_10_5V: now also U17.24 (2A10), U19.12 (1A10), U21.24 (2A10)
- net burst_11_5V: now also U15.2 (1A1), U19.13 (2A1), U22.2 (1A1)
- net burst_12_5V: now also U15.3 (1A2), U19.14 (2A2), U22.3 (1A2)
- net burst_13_5V: now also U15.4 (1A3), U19.16 (2A3), U22.4 (1A3)
- net burst_14_5V: now also U15.5 (1A4), U19.18 (2A4), U22.5 (1A4)
- net burst_15_5V: now also U15.6 (1A5), U19.19 (2A5), U22.6 (1A5)
- net burst_16_5V: now also U15.7 (1A6), U19.20 (2A6), U22.7 (1A6)
- net burst_17_5V: now also U15.9 (1A7), U19.21 (2A7), U22.9 (1A7)
- net burst_18_5V: now also U15.10 (1A8), U19.22 (2A8), U22.10 (1A8)
- net burst_19_5V: now also U15.11 (1A9), U19.23 (2A9), U22.11 (1A9)
- net burst_1_5V: now also U17.13 (2A1), U19.2 (1A1), U21.13 (2A1)
- net burst_20_5V: now also U15.12 (1A10), U19.24 (2A10), U22.12 (1A10)
- net burst_21_5V: now also U15.13 (2A1), U20.2 (1A1), U22.13 (2A1)
- net burst_22_5V: now also U15.14 (2A2), U20.3 (1A2), U22.14 (2A2)
- net burst_23_5V: now also U15.16 (2A3), U20.4 (1A3), U22.16 (2A3)
- net burst_24_5V: now also U15.18 (2A4), U20.5 (1A4), U22.18 (2A4)
- net burst_25_5V: now also U15.19 (2A5), U20.6 (1A5), U22.19 (2A5)
- net burst_26_5V: now also U15.20 (2A6), U20.7 (1A6), U22.20 (2A6)
- net burst_27_5V: now also U15.21 (2A7), U20.9 (1A7), U22.21 (2A7)
- net burst_28_5V: now also U15.22 (2A8), U20.10 (1A8), U22.22 (2A8)
- net burst_29_5V: now also U15.23 (2A9), U20.11 (1A9), U22.23 (2A9)
- net burst_2_5V: now also U17.14 (2A2), U19.3 (1A2), U21.14 (2A2)
- net burst_30_5V: now also U15.24 (2A10), U20.12 (1A10), U22.24 (2A10)
- net burst_31_5V: now also U18.2 (1A1), U20.13 (2A1), U23.2 (1A1)
- net burst_32_5V: now also U18.3 (1A2), U20.14 (2A2), U23.3 (1A2)
- net burst_33_5V: now also U18.4 (1A3), U20.16 (2A3), U23.4 (1A3)
- net burst_34_5V: now also U18.5 (1A4), U20.18 (2A4), U23.5 (1A4)
- net burst_35_5V: now also U18.6 (1A5), U20.19 (2A5), U23.6 (1A5)
- net burst_36_5V: now also U18.7 (1A6), U20.20 (2A6), U23.7 (1A6)
- net burst_37_5V: now also U18.9 (1A7), U20.21 (2A7), U23.9 (1A7)
- net burst_38_5V: now also U18.10 (1A8), U20.22 (2A8), U23.10 (1A8)
- net burst_39_5V: now also U18.11 (1A9), U20.23 (2A9), U23.11 (1A9)
- net burst_3_5V: now also U17.16 (2A3), U19.4 (1A3), U21.16 (2A3)
- net burst_40_5V: now also U18.12 (1A10), U20.24 (2A10), U23.12 (1A10)
- net burst_41_5V: now also U18.13 (2A1), U21.2 (1A1), U23.13 (2A1)
- net burst_42_5V: now also U18.14 (2A2), U21.3 (1A2), U23.14 (2A2)
- net burst_43_5V: now also U18.16 (2A3), U21.4 (1A3), U23.16 (2A3)
- net burst_44_5V: now also U18.18 (2A4), U21.5 (1A4), U23.18 (2A4)
- net burst_45_5V: now also U18.19 (2A5), U21.6 (1A5), U23.19 (2A5)
- net burst_46_5V: now also U18.20 (2A6), U21.7 (1A6), U23.20 (2A6)
- net burst_47_5V: now also U18.21 (2A7), U21.9 (1A7), U23.21 (2A7)
- net burst_48_5V: now also U18.22 (2A8), U21.10 (1A8), U23.22 (2A8)
- net burst_4_5V: now also U17.18 (2A4), U19.5 (1A4), U21.18 (2A4)
- net burst_5_5V: now also U17.19 (2A5), U19.6 (1A5), U21.19 (2A5)
- net burst_6_5V: now also U17.20 (2A6), U19.7 (1A6), U21.20 (2A6)
- net burst_7_5V: now also U17.21 (2A7), U19.9 (1A7), U21.21 (2A7)
- net burst_8_5V: now also U17.22 (2A8), U19.10 (1A8), U21.22 (2A8)
- net burst_9_5V: now also U17.23 (2A9), U19.11 (1A9), U21.23 (2A9)
- net VCC_5V: now reaches C61.1, U12.3 (VI)
- net VCC_5V: now also 23A1024/23LC1.8 (VCC), C16.2, C17.1, C18.1, C19.1, C20.2, C21.1, C48.2, R10.1, R11.2, R18.2, U1.20 (VCCB), U10.20 (VCCB), U11.20 (VCCB), U13.20 (VCCB), U14.15 (VCC), U16.15 (VCC), U17.15 (VCC), U5.20 (VCCB), U7.18 (AVCC), U8.20 (VCCB), U9.20 (VCCB), U15.15 (VCC), U18.15 (VCC), U19.15 (VCC), U20.15 (VCC), U21.15 (VCC), U22.15 (VCC), U23.15 (VCC)
- net at U5.11 (~{OE}): now also R38.1
- net INT_5V: now reaches U5.12 (B7)
- net INT_5V: now also U7.32 (PD2)
- net CTS_5V: now reaches U5.13 (B6)
- net CTS_5V: now also U7.9 (PD5)
- net RTS_5V: now reaches U5.14 (B5)
- net RTS_5V: now also U7.2 (PD4)
- net SRAM_CS_: now reaches U5.6 (A4)
- net SRAM_CS_: now also J5.2 (Pin_2)
- net RTS: now reaches U5.7 (A5)
- net RTS: now also U6.25 (PA2)
- net CTS: now reaches U5.8 (A6)
- net CTS: now also U6.26 (PA3)
- net INT: now reaches U5.9 (A7)
- net INT: now also U6.53 (PB14)
- net at U9.11 (~{OE}): now also R42.1
- net BUS_1_DETECT: now reaches U6.35 (PB0)
- net BUS_1_DETECT: now also R19.1, R20.1
- net BUS_2_DETECT: now reaches U6.36 (PB1)
- net BUS_2_DETECT: now also R16.1, R17.1
- net BUS_3_DETECT: now reaches U6.37 (PB2)
- net BUS_3_DETECT: now also R21.1, R22.1
- net BUS_4_DETECT: now reaches U6.52 (PB13)
- net BUS_4_DETECT: now also R23.1, R24.1
- net SRAM_CS: now reaches U6.71 (PA12)
- net SRAM_CS: now also J5.1 (Pin_1)
- net at U8.11 (~{OE}): now also R43.1
- net BURST_10.2: now reaches U17.25 (2B10)
- net BURST_10.2: now also J8.10 (Pin_10)
- net BURST_9.2: now reaches U17.26 (2B9)
- net BURST_9.2: now also J8.9 (Pin_9)
- net BURST_8.2: now reaches U17.27 (2B8)
- net BURST_8.2: now also J8.8 (Pin_8)
- net BURST_7.2: now reaches U17.28 (2B7)
- net BURST_7.2: now also J8.7 (Pin_7)
- net BURST_6.2: now reaches U17.29 (2B6)
- net BURST_6.2: now also J8.6 (Pin_6)
- net BURST_5.2: now reaches U17.30 (2B5)
- net BURST_5.2: now also J8.5 (Pin_5)
- net BURST_4.2: now reaches U17.31 (2B4)
- net BURST_4.2: now also J8.4 (Pin_4)
- net BURST_3.2: now reaches U17.33 (2B3)
- net BURST_3.2: now also J8.3 (Pin_3)
- net BURST_2.2: now reaches U17.34 (2B2)
- net BURST_2.2: now also J8.2 (Pin_2)
- net BURST_1.2: now reaches U17.35 (2B1)
- net BURST_1.2: now also J8.1 (Pin_1)
- net at U10.11 (~{OE}): now also R41.1
- net at U1.11 (~{OE}): now also R44.1
- net at U13.11 (~{OE}): now also R39.1
- net at U11.11 (~{OE}): now also R40.1
- net VCC_3: no longer names the net of J4.50 (Pin_50)
- net VCC_3: now also R19.2
- new net: J9.50 (Pin_50), R21.2
- new net: J8.50 (Pin_50), R17.2
- new net: J10.50 (Pin_50), R23.2
- new net BURST_1.3: J9.1 (Pin_1), U19.46 (1B1)
- new net BURST_1.4: J10.1 (Pin_1), U21.35 (2B1)
- new net BURST_10.3: J9.10 (Pin_10), U19.36 (1B10)
- new net BURST_10.4: J10.10 (Pin_10), U21.25 (2B10)
- new net BURST_11.2: J8.11 (Pin_11), U15.46 (1B1)
- new net BURST_11.3: J9.11 (Pin_11), U19.35 (2B1)
- new net BURST_11.4: J10.11 (Pin_11), U22.46 (1B1)
- new net BURST_12.2: J8.12 (Pin_12), U15.45 (1B2)
- new net BURST_12.3: J9.12 (Pin_12), U19.34 (2B2)
- new net BURST_12.4: J10.12 (Pin_12), U22.45 (1B2)
- new net BURST_13.2: J8.13 (Pin_13), U15.44 (1B3)
- new net BURST_13.3: J9.13 (Pin_13), U19.33 (2B3)
- new net BURST_13.4: J10.13 (Pin_13), U22.44 (1B3)
- new net BURST_14.2: J8.14 (Pin_14), U15.43 (1B4)
- new net BURST_14.3: J9.14 (Pin_14), U19.31 (2B4)
- new net BURST_14.4: J10.14 (Pin_14), U22.43 (1B4)
- new net BURST_15.2: J8.15 (Pin_15), U15.42 (1B5)
- new net BURST_15.3: J9.15 (Pin_15), U19.30 (2B5)
- new net BURST_15.4: J10.15 (Pin_15), U22.42 (1B5)
- new net BURST_16.2: J8.16 (Pin_16), U15.40 (1B6)
- new net BURST_16.3: J9.16 (Pin_16), U19.29 (2B6)
- new net BURST_16.4: J10.16 (Pin_16), U22.40 (1B6)
- new net BURST_17.2: J8.17 (Pin_17), U15.39 (1B7)
- new net BURST_17.3: J9.17 (Pin_17), U19.28 (2B7)
- new net BURST_17.4: J10.17 (Pin_17), U22.39 (1B7)
- new net BURST_18.2: J8.18 (Pin_18), U15.38 (1B8)
- new net BURST_18.3: J9.18 (Pin_18), U19.27 (2B8)
- new net BURST_18.4: J10.18 (Pin_18), U22.38 (1B8)
- new net BURST_19.2: J8.19 (Pin_19), U15.37 (1B9)
- new net BURST_19.3: J9.19 (Pin_19), U19.26 (2B9)
- new net BURST_19.4: J10.19 (Pin_19), U22.37 (1B9)
- new net BURST_2.3: J9.2 (Pin_2), U19.45 (1B2)
- new net BURST_2.4: J10.2 (Pin_2), U21.34 (2B2)
- new net BURST_20.2: J8.20 (Pin_20), U15.36 (1B10)
- new net BURST_20.3: J9.20 (Pin_20), U19.25 (2B10)
- new net BURST_20.4: J10.20 (Pin_20), U22.36 (1B10)
- new net BURST_21.2: J8.21 (Pin_21), U15.35 (2B1)
- new net BURST_21.3: J9.21 (Pin_21), U20.46 (1B1)
- new net BURST_21.4: J10.21 (Pin_21), U22.35 (2B1)
- new net BURST_22.2: J8.22 (Pin_22), U15.34 (2B2)
- new net BURST_22.3: J9.22 (Pin_22), U20.45 (1B2)
- new net BURST_22.4: J10.22 (Pin_22), U22.34 (2B2)
- new net BURST_23.2: J8.23 (Pin_23), U15.33 (2B3)
- new net BURST_23.3: J9.23 (Pin_23), U20.44 (1B3)
- new net BURST_23.4: J10.23 (Pin_23), U22.33 (2B3)
- new net BURST_24.2: J8.24 (Pin_24), U15.31 (2B4)
- new net BURST_24.3: J9.24 (Pin_24), U20.43 (1B4)
- new net BURST_24.4: J10.24 (Pin_24), U22.31 (2B4)
- new net BURST_25.2: J8.25 (Pin_25), U15.30 (2B5)
- new net BURST_25.3: J9.25 (Pin_25), U20.42 (1B5)
- new net BURST_25.4: J10.25 (Pin_25), U22.30 (2B5)
- new net BURST_26.2: J8.26 (Pin_26), U15.29 (2B6)
- new net BURST_26.3: J9.26 (Pin_26), U20.40 (1B6)
- new net BURST_26.4: J10.26 (Pin_26), U22.29 (2B6)
- new net BURST_27.2: J8.27 (Pin_27), U15.28 (2B7)
- new net BURST_27.3: J9.27 (Pin_27), U20.39 (1B7)
- new net BURST_27.4: J10.27 (Pin_27), U22.28 (2B7)
- new net BURST_28.2: J8.28 (Pin_28), U15.27 (2B8)
- new net BURST_28.3: J9.28 (Pin_28), U20.38 (1B8)
- new net BURST_28.4: J10.28 (Pin_28), U22.27 (2B8)
- new net BURST_29.2: J8.29 (Pin_29), U15.26 (2B9)
- new net BURST_29.3: J9.29 (Pin_29), U20.37 (1B9)
- new net BURST_29.4: J10.29 (Pin_29), U22.26 (2B9)
- new net BURST_3.3: J9.3 (Pin_3), U19.44 (1B3)
- new net BURST_3.4: J10.3 (Pin_3), U21.33 (2B3)
- new net BURST_30,3: J9.30 (Pin_30)
- new net BURST_30.2: J8.30 (Pin_30), U15.25 (2B10)
- new net BURST_30.3: U20.36 (1B10)
- new net BURST_30.4: J10.30 (Pin_30), U22.25 (2B10)
- new net BURST_31.2: J8.31 (Pin_31), U18.46 (1B1)
- new net BURST_31.3: J9.31 (Pin_31), U20.35 (2B1)
- new net BURST_31.4: J10.31 (Pin_31), U23.46 (1B1)
- new net BURST_32.2: J8.32 (Pin_32), U18.45 (1B2)
- new net BURST_32.3: J9.32 (Pin_32), U20.34 (2B2)
- new net BURST_32.4: J10.32 (Pin_32), U23.45 (1B2)
- new net BURST_33.2: J8.33 (Pin_33), U18.44 (1B3)
- new net BURST_33.3: J9.33 (Pin_33), U20.33 (2B3)
- new net BURST_33.4: J10.33 (Pin_33), U23.44 (1B3)
- new net BURST_34.2: J8.34 (Pin_34), U18.43 (1B4)
- new net BURST_34.3: J9.34 (Pin_34), U20.31 (2B4)
- new net BURST_34.4: J10.34 (Pin_34), U23.43 (1B4)
- new net BURST_35.2: J8.35 (Pin_35), U18.42 (1B5)
- new net BURST_35.3: J9.35 (Pin_35), U20.30 (2B5)
- new net BURST_35.4: J10.35 (Pin_35), U23.42 (1B5)
- new net BURST_36.2: J8.36 (Pin_36), U18.40 (1B6)
- new net BURST_36.3: J9.36 (Pin_36), U20.29 (2B6)
- new net BURST_36.4: J10.36 (Pin_36), U23.40 (1B6)
- new net BURST_37.2: J8.37 (Pin_37), U18.39 (1B7)
- new net BURST_37.3: J9.37 (Pin_37), U20.28 (2B7)
- new net BURST_37.4: J10.37 (Pin_37), U23.39 (1B7)
- new net BURST_38.2: J8.38 (Pin_38), U18.38 (1B8)
- new net BURST_38.3: J9.38 (Pin_38), U20.27 (2B8)
- new net BURST_38.4: J10.38 (Pin_38), U23.38 (1B8)
- new net BURST_39.2: J8.39 (Pin_39), U18.37 (1B9)
- new net BURST_39.3: J9.39 (Pin_39), U20.26 (2B9)
- new net BURST_39.4: J10.39 (Pin_39), U23.37 (1B9)
- new net BURST_4.3: J9.4 (Pin_4), U19.43 (1B4)
- new net BURST_4.4: J10.4 (Pin_4), U21.31 (2B4)
- new net BURST_40.2: J8.40 (Pin_40), U18.36 (1B10)
- new net BURST_40.3: J9.40 (Pin_40), U20.25 (2B10)
- new net BURST_40.4: J10.40 (Pin_40), U23.36 (1B10)
- new net BURST_41.2: J8.41 (Pin_41), U18.35 (2B1)
- new net BURST_41.3: J9.41 (Pin_41), U21.46 (1B1)
- new net BURST_41.4: J10.41 (Pin_41), U23.35 (2B1)
- new net BURST_42.2: J8.42 (Pin_42), U18.34 (2B2)
- new net BURST_42.3: J9.42 (Pin_42), U21.45 (1B2)
- new net BURST_42.4: J10.42 (Pin_42), U23.34 (2B2)
- new net BURST_43.2: J8.43 (Pin_43), U18.33 (2B3)
- new net BURST_43.3: J9.43 (Pin_43), U21.44 (1B3)
- new net BURST_43.4: J10.43 (Pin_43), U23.33 (2B3)
- new net BURST_44.2: J8.44 (Pin_44), U18.31 (2B4)
- new net BURST_44.3: J9.44 (Pin_44), U21.43 (1B4)
- new net BURST_44.4: J10.44 (Pin_44), U23.31 (2B4)
- new net BURST_45.2: J8.45 (Pin_45), U18.30 (2B5)
- new net BURST_45.3: J9.45 (Pin_45), U21.42 (1B5)
- new net BURST_45.4: J10.45 (Pin_45), U23.30 (2B5)
- new net BURST_46.2: J8.46 (Pin_46), U18.29 (2B6)
- new net BURST_46.3: J9.46 (Pin_46), U21.40 (1B6)
- new net BURST_46.4: J10.46 (Pin_46), U23.29 (2B6)
- new net BURST_47.2: J8.47 (Pin_47), U18.28 (2B7)
- new net BURST_47.3: J9.47 (Pin_47), U21.39 (1B7)
- new net BURST_47.4: J10.47 (Pin_47), U23.28 (2B7)
- new net BURST_48.2: J8.48 (Pin_48), U18.27 (2B8)
- new net BURST_48.3: J9.48 (Pin_48), U21.38 (1B8)
- new net BURST_48.4: J10.48 (Pin_48), U23.27 (2B8)
- new net BURST_5.3: J9.5 (Pin_5), U19.42 (1B5)
- new net BURST_5.4: J10.5 (Pin_5), U21.30 (2B5)
- new net BURST_6.3: J9.6 (Pin_6), U19.40 (1B6)
- new net BURST_6.4: J10.6 (Pin_6), U21.29 (2B6)
- new net BURST_7.3: J9.7 (Pin_7), U19.39 (1B7)
- new net BURST_7.4: J10.7 (Pin_7), U21.28 (2B7)
- new net BURST_8.3: J9.8 (Pin_8), U19.38 (1B8)
- new net BURST_8.4: J10.8 (Pin_8), U21.27 (2B8)
- new net BURST_9.3: J9.9 (Pin_9), U19.37 (1B9)
- new net BURST_9.4: J10.9 (Pin_9), U21.26 (2B9)
- no-connect marks 13 -> 5
Other:
- moved on the sheet: J1, J12, J4, U14, U16, U5

Commit message: .
Parts:
- removed R26, R27, R30, R31, R33, R34, R36, R37: 10k, Resistor_SMD:R_0402_1005Metric, symbol Device:R
Connections:
- net BUS_1: no longer U6.67 (PA8)
- net BUS_1_DETECT: no longer U6.35 (PB0)
- net BUS_2: no longer U6.68 (PA9)
- net BUS_2_DETECT: no longer U6.36 (PB1)
- net BUS_3: no longer U6.69 (PA10)
- net BUS_3_DETECT: no longer U6.37 (PB2)
- net BUS_4: no longer U6.70 (PA11)
- net BUS_4_DETECT: no longer U6.52 (PB13)
- net CTS: no longer U6.26 (PA3)
- net INT: no longer U6.53 (PB14)
- net J_C: no longer U6.51 (PB12)
- net RTS: no longer U6.25 (PA2)
- net SRAM_CS: no longer U6.71 (PA12)
- net burst_1: now also U6.80 (PC12); no longer U6.15 (PC0)
- net burst_10: now also U6.65 (PC8); no longer U6.66 (PC9)
- net burst_11: now also U6.64 (PC7); no longer U6.78 (PC10)
- net burst_12: now also U6.63 (PC6); no longer U6.79 (PC11)
- net burst_13: now also U6.62 (PD15); no longer U6.80 (PC12)
- net burst_14: now also U6.61 (PD14); no longer U6.7 (PC13)
- net burst_15: now also U6.60 (PD13); no longer U6.8 (PC14)
- net burst_16: now also U6.59 (PD12); no longer U6.9 (PC15)
- net burst_17: now also U6.58 (PD11); no longer U6.54 (PB15)
- net burst_18: now also U6.57 (PD10); no longer U6.97 (PE0)
- net burst_19: now also U6.56 (PD9); no longer U6.1 (PE2)
- net burst_2: now also U6.79 (PC11); no longer U6.16 (PC1)
- net burst_20: now also U6.55 (PD8); no longer U6.2 (PE3)
- net burst_21: now also U6.54 (PB15); no longer U6.3 (PE4)
- net burst_22: now also U6.53 (PB14); no longer U6.4 (PE5)
- net burst_23: now also U6.52 (PB13); no longer U6.5 (PE6)
- net burst_24: now also U6.51 (PB12); no longer U6.38 (PE7)
- net burst_25: now also U6.46 (PE15); no longer U6.39 (PE8)
- net burst_26: now also U6.45 (PE14); no longer U6.40 (PE9)
- net burst_27: now also U6.44 (PE13); no longer U6.41 (PE10)
- net burst_28: now also U6.43 (PE12); no longer U6.42 (PE11)
- net burst_29: now also U6.42 (PE11); no longer U6.43 (PE12)
- net burst_3: now also U6.78 (PC10); no longer U6.17 (PC2)
- net burst_30: now also U6.41 (PE10); no longer U6.44 (PE13)
- net burst_31: now also U6.40 (PE9); no longer U6.45 (PE14)
- net burst_32: now also U6.39 (PE8); no longer U6.46 (PE15)
- net burst_33: now also U6.38 (PE7); no longer U6.81 (PD0)
- net burst_34: now also U6.37 (PB2); no longer U6.82 (PD1)
- net burst_35: now also U6.36 (PB1); no longer U6.83 (PD2)
- net burst_36: now also U6.35 (PB0); no longer U6.84 (PD3)
- net burst_37: now also U6.34 (PC5); no longer U6.85 (PD4)
- net burst_38: now also U6.33 (PC4); no longer U6.86 (PD5)
- net burst_39: now also U6.26 (PA3); no longer U6.87 (PD6)
- net burst_4: now also U6.71 (PA12); no longer U6.18 (PC3)
- net burst_40: now also U6.25 (PA2); no longer U6.88 (PD7)
- net burst_41: now also U6.81 (PD0); no longer U6.55 (PD8)
- net burst_42: now also U6.82 (PD1); no longer U6.56 (PD9)
- net burst_43: now also U6.83 (PD2); no longer U6.57 (PD10)
- net burst_44: now also U6.84 (PD3); no longer U6.58 (PD11)
- net burst_45: now also U6.85 (PD4); no longer U6.59 (PD12)
- net burst_46: now also U6.86 (PD5); no longer U6.60 (PD13)
- net burst_47: now also U6.87 (PD6); no longer U6.61 (PD14)
- net burst_48: now also U6.88 (PD7); no longer U6.62 (PD15)
- net burst_5: now also U6.70 (PA11); no longer U6.33 (PC4)
- net burst_6: now also U6.69 (PA10); no longer U6.34 (PC5)
- net burst_7: now also U6.68 (PA9); no longer U6.63 (PC6)
- net burst_8: now also U6.67 (PA8); no longer U6.64 (PC7)
- net burst_9: now also U6.66 (PC9); no longer U6.65 (PC8)

Commit message: .
Parts:
- removed C1_Crystal1, C2_Crystal1: C_Small, Capacitor_THT:CP_Radial_D5.0mm_P2.50mm, symbol Device:C_Small
- added 220UF1, 220UF2: C_Polarized, Capacitor_THT:C_Disc_D3.0mm_W1.6mm_P2.50mm, symbol Device:C_Polarized
- added C22, C23: 10p, Capacitor_SMD:C_0402_1005Metric, symbol Device:C
- added C24, C25, C26, C27, C29, C30, C32, C34, C36, C38, C41, C43, C49, C51, C53, C55, C57, C59, C64, C66, C67: 100n, Capacitor_SMD:C_0402_1005Metric, symbol Device:C
- added C31, C33, C35, C37, C39, C42, C45, C50, C52, C54, C56, C58: 2.2u, Capacitor_SMD:C_0402_1005Metric, symbol Device:C
- added C4321: 16PK4700MEFC12.5X25, symbol Device:C_Polarized
- added C4322: T520Y337M006ATE040, symbol Device:C_Small
- added C60, C63: 47pf, Capacitor_SMD:C_0402_1005Metric, symbol Device:C
- added C65: 4.7u, Capacitor_SMD:C_0603_1608Metric, symbol Device:C
- added D1, D2, D7: LED, LED_SMD:LED_0603_1608Metric, symbol Device:LED
- added J15: PJ-102A, Connector_BarrelJack:BarrelJack_Horizontal, symbol dk_Barrel-Power-Connectors:PJ-102A
- added J6: USB_A, Connector_USB:USB_B_Lumberg_2411_02_Horizontal, symbol Connector:USB_A
- added R26: 4k7, Resistor_SMD:R_0402_1005Metric, symbol Device:R
- added R27, R33: 10k, Resistor_SMD:R_0402_1005Metric, symbol Device:R
- added R30, R31, R34: 200, Resistor_SMD:R_0402_1005Metric, symbol Device:R
- added SW5: SW_Push, Button_Switch_THT:SW_PUSH_1P1T_6x3.5mm_H4.3_APEM_MJTP1243, symbol Switch:SW_Push
- added U3: FT232RL, Package_SO:SSOP-28_5.3x10.2mm_P0.65mm, symbol Interface_USB:FT232RL
Connections:
- net AT_CS: now also J12.5 (Pin_5)
- net AT_MISO: now also J12.9 (Pin_9)
- net AT_MOSI: now also J12.1 (Pin_1)
- net AT_SCK: now also J12.7 (Pin_7)
- net CS: no longer J12.5 (Pin_5)
- net GND: now also 220UF1.2, 220UF2.2, C22.1, C23.2, C24.2, C25.2, C26.2, C27.2, C29.2, C30.2, C31.2, C32.2, C33.2, C34.2, C35.2, C36.2, C37.2, C38.2, C39.2, C41.2, C42.2, C43.2, C4321.2, C4322.1, C45.2, C49.2, C50.2, C51.2, C52.2, C53.2, C54.2, C55.2, C56.2, C57.2, C58.2, C59.2, C60.2, C63.2, C64.1, C65.1, C66.1, C67.1, J15.2, J15.3, J6.4 (GND), R27.1, R34.1, SW5.2, U3.18 (GND), U3.21 (GND), U3.25 (AGND), U3.26 (TEST), U3.7 (GND)
- net MISO: no longer J12.9 (Pin_9)
- net MOSI: no longer J12.1 (Pin_1)
- net SCK: no longer J12.7 (Pin_7)
- net VCC: now also C31.1, C32.1, C37.1, C38.1, C42.1, C43.1, C50.1, C51.1, C54.1, C55.1, C58.1, C59.1; no longer U7.20 (AREF)
- net VCC_5V: now also U7.20 (AREF), 220UF1.1, 220UF2.1, C33.1, C34.1, C35.1, C36.1, C39.1, C41.1, C4321.1, C4322.2, C45.1, C49.1, C52.1, C53.1, C56.1, C57.1, C65.2, C66.2, C67.2, D2.2 (A), J15.1, R30.1, R31.1, R33.1, U3.20 (VCC), U3.4 (VCCIO)
- net at R41.1, U10.11 (~{OE}): now also C27.1
- net at R42.1, U9.11 (~{OE}): now also C26.1
- net at R44.1, U1.11 (~{OE}): now also C25.1
- net at U7.8 (XTAL2/PB7), Y2.1: now also C23.1
- net at R43.1, U8.11 (~{OE}): now also C24.1
- net at U7.7 (XTAL1/PB6), Y2.2: now also C22.2
- net at R39.1, U13.11 (~{OE}): now also C30.1
- net at R40.1, U11.11 (~{OE}): now also C29.1
- new net: D1.2 (A), R30.2
- new net: R26.1, R27.2, SW5.1, U3.19 (~{RESET})
- new net: R33.2, U3.14 (CBUS3)
- new net: J6.1 (VBUS), R26.2
- new net: D7.2 (A), R31.2
- new net: D1.1 (K), U3.13 (CBUS2)
- new net: D2.1 (K), R34.2
- new net: C64.2, U3.17 (3V3OUT)
- new net: D7.1 (K), U3.22 (CBUS1)
- new net D+: C63.1, J6.3 (D+), U3.15 (USBD+)
- new net D-: C60.1, J6.2 (D-), U3.16 (USBD-)
- new net RXD_CONV: U3.5 (RXD)
- new net TXD_CONV: U3.1 (TXD)
- no-connect marks 5 -> 18
Other:
- moved on the sheet: R39, R40, R41, R42, R43, R44

Commit message: .
Parts:
- C4321: footprint (none) -> Capacitor_THT:CP_Radial_D5.0mm_P2.50mm
- C4322: footprint (none) -> Capacitor_SMD:CP_Elec_10x10
- J5: footprint Connector_PinSocket_2.54mm:PinSocket_1x01_P2.54mm_Vertical -> Connector_PinSocket_2.54mm:PinSocket_1x02_P2.54mm_Vertical
- SPEAKER1: footprint (none) -> Connector_JST:JST_EH_B3B-EH-A_1x03_P2.50mm_Vertical
- V_1, V_2, V_3, V_4: footprint Connector_PinHeader_2.54mm:PinHeader_1x02_P2.54mm_Vertical -> Connector_JST:JST_EH_B2B-EH-A_1x02_P2.50mm_Vertical
Connections:
- net 3.3V is gone; now on net VCC: JTAG1.1 (Pin_1), JTAG1.2 (Pin_2)
- net RXD_CONV is gone; now on net TX: U3.5 (RXD)
- net TXD_CONV is gone; now on net RX: U3.1 (TXD)
- net BUS_1: now also U6.96 (PB9)
- net BUS_1_DETECT: now also U6.4 (PE5)
- net BUS_2: now also U6.1 (PE2)
- net BUS_2_DETECT: now also U6.5 (PE6)
- net BUS_3: now also U6.2 (PE3)
- net BUS_3_DETECT: now also U6.97 (PE0)
- net BUS_4: now also U6.3 (PE4)
- net BUS_4_DETECT: now also U6.47 (PB10)
- net CTS: now also U6.92 (PB6)
- net INT: now also U6.95 (PB8)
- net J_A: now also U6.8 (PC14); no longer U6.96 (PB9)
- net J_B: now also U6.9 (PC15); no longer U6.47 (PB10)
- net J_C: now also U6.7 (PC13)
- net J_DOWN: now also U6.16 (PC1); no longer U6.92 (PB6)
- net J_LEFT: now also U6.17 (PC2); no longer U6.93 (PB7)
- net J_RIGHT: now also U6.18 (PC3); no longer U6.95 (PB8)
- net J_UP: now also U6.15 (PC0); no longer U6.91 (PB5)
- net RTS: now also U6.91 (PB5)
- net SRAM_CS: now also U6.93 (PB7)
- net VCC_5V: now also Q1.3 (D), Q2.3 (D), Q3.3 (D), Q4.3 (D), U7.4 (VCC), U7.6 (VCC)

Commit message: .
Parts:
- added ATUART1: Conn_01x03_Pin, Connector_JST:JST_EH_B3B-EH-A_1x03_P2.50mm_Vertical, symbol Connector:Conn_01x03_Pin
- added LCD1: Conn_01x04_Pin, Connector_JST:JST_EH_B4B-EH-A_1x04_P2.50mm_Vertical, symbol Connector:Conn_01x04_Pin
- renumbered SW3 to ATRESET1, SW1 to BOOT0, SW5 to FRESET1, D7 to FRX1, D1 to FTX1, J4 to GRID1, J8 to GRID2, J9 to GRID3, J10 to GRID4, D2 to PWR1, SW2 to STRESET1, J1 to STUART1, J12 to USBASP1
Connections:
- net BURST_30,3 is gone; now on net BURST_30.3: GRID3.30 (Pin_30)
- net AT_MISO: now also 23A1024/23LC1.2 (SO/SIO1); no longer 23A1024/23LC1.5 (SI/SIO0)
- net AT_MOSI: now also 23A1024/23LC1.5 (SI/SIO0); no longer 23A1024/23LC1.2 (SO/SIO1)
- net AT_RX: now also ATUART1.1 (Pin_1)
- net AT_TX: now also ATUART1.2 (Pin_2)
- net GND: now also ATUART1.3 (Pin_3), LCD1.4 (Pin_4)
- net SCL: now also LCD1.1 (Pin_1)
- net SDA: now also LCD1.2 (Pin_2)
- net VCC_5V: now also LCD1.3 (Pin_3)
- net burst_1 renamed burst_1_
- net burst_10 renamed burst_10_
- net burst_11 renamed burst_11_
- net burst_12 renamed burst_12_
- net burst_13 renamed burst_13_
- net burst_14 renamed burst_14_
- net burst_15 renamed burst_15_
- net burst_16 renamed burst_16_
- net burst_17 renamed burst_17_
- net burst_18 renamed burst_18_
- net burst_19 renamed burst_19_
- net burst_2 renamed burst_2_
- net burst_20 renamed burst_20_
- net burst_21 renamed burst_21_
- net burst_22 renamed burst_22_
- net burst_23 renamed burst_23_
- net burst_24 renamed burst_24_
- net burst_25 renamed burst_25_
- net burst_26 renamed burst_26_
- net burst_27 renamed burst_27_
- net burst_28 renamed burst_28_
- net burst_29 renamed burst_29_
- net burst_3 renamed burst_3_
- net burst_30 renamed burst_30_
- net burst_31 renamed burst_31_
- net burst_32 renamed burst_32_
- net burst_33 renamed burst_33_
- net burst_34 renamed burst_34_
- net burst_35 renamed burst_35_
- net burst_36 renamed burst_36_
- net burst_37 renamed burst_37_
- net burst_38 renamed burst_38_
- net burst_39 renamed burst_39_
- net burst_4 renamed burst_4_
- net burst_40 renamed burst_40_
- net burst_41 renamed burst_41_
- net burst_42 renamed burst_42_
- net burst_43 renamed burst_43_
- net burst_44 renamed burst_44_
- net burst_45 renamed burst_45_
- net burst_46 renamed burst_46_
- net burst_47 renamed burst_47_
- net burst_48 renamed burst_48_
- net burst_5 renamed burst_5_
- net burst_6 renamed burst_6_
- net burst_7 renamed burst_7_
- net burst_8 renamed burst_8_
- net burst_9 renamed burst_9_
- no-connect marks 18 -> 34
